File: ADC.sch (EAGLE design)
At the start: 40 parts, among them IC1 AD8221ARZ, IC2 TLC2254ID, Q1 8MHz

Commit message: .
Parts:
- removed U$1: ADS1256IDBT, nanoeeg:ADS1256IDBT
- added C14: 4n7, rcl:C-EUC0805
- added C15, C16, C17, C18: 0.1, rcl:C-EUC0805
- added DC1: TMV0505D, dc-dc-converter:NMA
- added IC3: ADS1256IDBT, nanoeeg:ADS1256IDBT
- added IC4: AD8605ARTZ, nanoeeg:AD8605ARTZ
- added IC5: TS5A23157DGSR, nanoeeg:TS5A23157DGSR
- added IC6: ADUM1402ARWZ, nanoeeg:ADUM1402ARWZ
- added INT: (no value), pinhead:PINHD-1X8
- added R18, R20: 10K, rcl:R-EU_R0805
- added R19: 40K, rcl:R-EU_R0805
- added R21: 124K, rcl:R-EU_R0805
- added R22, R23, R25: 1K, rcl:R-EU_R0805
- added R24: 3K, rcl:R-EU_R0805
Connections:
- removed net N$18 (its old number): C12.2, C13.1, R12.2
- new net CH1SW1: IC2.OUT2, IC5.NC1, R11.1, R12.2, R19.2
- new net CH1SW2: IC5.COM1, R19.1, R20.2
- new net CH2SW1: IC5.NC2
- new net CH2SW2: IC5.COM2
- new net N$15: C13.2, IC2.+IN2, R13.1
- new net N$16: IC2.-IN2, R10.2, R11.2
- new net N$17: C12.2, C13.1, R12.1
- new net N$28: C14.2, IC2.OUT1, R21.1, R22.2
- new net N$29: C14.1, IC2.-IN1, R20.1, R21.2
- new net N$30: IC4.-IN, R22.1, R25.1
- new net N$31: IC3.D0/CLKOUT, IC5.IN1, IC5.IN2
- new net N$32: IC6.VIA, R14.2
- new net N$33: IC6.VIB, R17.2
- new net N$34: IC6.VOC, R15.2
- new net N$35: IC6.VOD, R16.2
- new net N$36: DC1.+VIN, INT.1
- new net N$37: C18.2, DC1.-VIN, IC6.GND2, IC6.GND2_, INT.3, INT.8
- new net N$38: C18.1, IC6.VDD2, IC6.VE2, INT.2
- new net N$40: IC6.VID, INT.7
- new net N$41: IC6.VIC, INT.6
- new net N$42: IC6.VOB, INT.5
- new net N$43: IC6.VOA, INT.4
- new net VREF: C16.1, IC3.VREFP, R24.1
- net +3.3V: now also C17.1, IC3.DVDD, IC3.RESET, IC3.SYNC/PDWN, IC5.VCC, IC6.VDD1, IC6.VE1; no longer U$1.DVDD, U$1.RESET, U$1.SYNC/PDWN
- net +5VA: now also C15.1, IC3.AVDD, IC4.+VS; no longer U$1.AVDD
- net GND: now also C15.2, C16.2, C17.2, DC1.COM, IC3.AGND, IC3.CS, IC3.DGND, IC3.VREFN, IC4.-VS, IC5.GND, IC6.GND1, IC6.GND1_, R13.2, R18.1, R23.2; no longer R13.1, U$1.AGND, U$1.DGND
- net N$11: now also IC3.DRDY; no longer U$1.DRDY
- net N$12: now also IC3.XTAL2; no longer U$1.XTAL2
- net N$13: now also IC3.XTAL1/CLKIN; no longer U$1.XTAL1/CLKIN
- net N$14: now also IC3.SCLK; no longer U$1.SCLK
- net N$19: now also IC4.+IN, R23.1, R24.2; no longer IC2.OUT1, R11.1, R12.1
- net N$20: now also R18.2; no longer C13.2, R13.2
- net N$21: now also IC3.AIN0, IC4.OUT, R25.2; no longer IC2.-IN1, R10.2, R11.2
- net N$22: now also IC3.DIN; no longer U$1.DIN
- net N$23: now also IC3.DOUT; no longer U$1.DOUT
Other:
- moved on the sheet: C10, C12, C13, C7, C8, C9, Q1, R10, R11, R12, R13, R14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

Commit message: Circuit alpha version; routing in progress
Parts:
- removed DC1: TMV0505D, dc-dc-converter:NMA
- added C100, C114, C128, C41, C58, C72, C86: 47n, rcl:C-EUC0805
- added C101, C115, C129, C42, C56, C59, C73, C87: 33n, rcl:C-EUC0805
- added C102, C106, C107, C108, C109, C112, C113, C116, C120, C121, C122, C123, C126, C127, C130, C19, C24, C25, C26, C28, C33, C34, C35, C36, C39, C40, C43, C44, C48, C49, C50, C51, C52, C55, C57, C60, C64, C65, C66, C67, C70, C71, C74, C78, C79, C80, C81, C84, C85, C88, C92, C93, C94, C95, C98, C99: 0.1, rcl:C-EUC0805
- added C103, C117, C30, C45, C61, C75, C89: 10pF, rcl:C-EUC0805
- added C104, C105, C118, C119, C31, C32, C46, C47, C62, C63, C76, C77, C90, C91: 100pF, rcl:C-EUC0805
- added C110, C111, C124, C125, C37, C38, C53, C54, C68, C69, C82, C83, C96, C97: 1u, rcl:C-EUC0805
- added C20, C21, C22, C23, C27, C29: 47u, rcl:CPOL-EUE2-4
- added D10, D11, D12, D13, D14, D15, D16, D17, D18, D19, D20, D21, D22, D23, D24, D25, D26, D27, D28, D29, D30, D31, D32, D5, D6, D7, D8, D9: BAV199, diode:BAV199
- added G1: TMV0505D, nanoeeg:TMV0505D
- added IC10, IC13, IC16, IC19, IC22, IC25, IC28: AD8605ARTZ, nanoeeg:AD8605ARTZ
- added IC11, IC14, IC17, IC20, IC23, IC26, IC8: AD8221ARZ, nanoeeg:AD8221ARZ
- added IC12, IC15, IC18, IC21, IC24, IC27, IC9: TLC2254ID, nanoeeg:TLC2254ID
- added IC7: REF3125AIDBZT, nanoeeg:REF3125AIDBZT
- added IN2: IN2, pinhead:PINHD-1X4
- added IN3: IN3, pinhead:PINHD-1X4
- added IN4: IN4, pinhead:PINHD-1X4
- added IN5: IN5, pinhead:PINHD-1X4
- added IN6: IN6, pinhead:PINHD-1X4
- added IN7: IN7, pinhead:PINHD-1X4
- added IN8: IN8, pinhead:PINHD-1X4
- added L1, L2: 100uH, rcl:L-USL4532P
- added R100, R119, R120, R139, R140, R159, R160, R39, R40, R59, R60, R79, R80, R99: 1K, rcl:R-EU_R0805
- added R101, R102, R103, R112, R113, R114, R117, R118, R121, R122, R123, R132, R133, R134, R137, R138, R141, R142, R143, R152, R153, R154, R157, R158, R161, R162, R163, R32, R33, R34, R37, R38, R41, R42, R43, R52, R53, R54, R57, R58, R61, R62, R63, R72, R73, R74, R77, R78, R81, R82, R83, R92, R93, R94, R97, R98: 100K, rcl:R-EU_R0805
- added R104, R107, R108, R124, R127, R128, R144, R147, R148, R164, R27, R28, R44, R47, R48, R64, R67, R68, R84, R87, R88: 100, rcl:R-EU_R0805
- added R105, R106, R109, R110, R125, R126, R129, R130, R145, R146, R149, R150, R26, R29, R30, R45, R46, R49, R50, R65, R66, R69, R70, R85, R86, R89, R90: 2K2, rcl:R-EU_R0805
- added R111, R131, R151, R31, R51, R71, R91: 2K, rcl:R-EU_R0805
- added R115, R135, R155, R35, R55, R75, R95: 910K, rcl:R-EU_R0805
- added R116, R136, R156, R36, R56, R76, R96: 680K, rcl:R-EU_R0805
- C10, C9: value 10pF -> 18p
- C12, C13: value 1 -> 1u
- C14: value 4n7 -> 47n
- COM: value (none) -> COM
- IC5: value TS5A23157DGSR -> MCP170333MB; device nanoeeg:TS5A23157DGSR -> linear:MCP170333MB
- IN1: value (none) -> IN1
- INT: value (none) -> INT
- R18: value 10K -> 100
- R19: value 40K -> 100K
- R20: value 10K -> 100K
- R21: value 124K -> 100K
- R23: value 1K -> 100K
- R24: value 3K -> 2K2
Connections:
- removed net CH2SW1: IC5.NC2
- removed net CH2SW2: IC5.COM2
- new net CH1SW3: IC12.OUT2, R55.1, R56.2, R58.2
- new net CH1SW4: IC15.OUT2, R75.1, R76.2, R78.2
- new net CH1SW5: IC18.OUT2, R95.1, R96.2, R98.2
- new net CH1SW6: IC21.OUT2, R115.1, R116.2, R118.2
- new net CH1SW7: IC24.OUT2, R135.1, R136.2, R138.2
- new net CH1SW8: IC27.OUT2, R155.1, R156.2, R158.2
- new net N$100: IC14.-RG, IC15.+IN3, R71.2
- new net N$101: IC14.+RG, IC15.+IN4, R71.1
- new net N$102: IC14.+IN, R70.2
- new net N$103: D16.AC, IC15.-IN4, IC15.OUT4, R68.2, R73.1
- new net N$104: D15.AC, IC15.-IN3, IC15.OUT3, R67.2, R72.1
- new net N$105: C69.2, IC15.+IN2, R77.1
- new net N$106: IC15.-IN2, R74.2, R75.2
- new net N$107: C68.2, C69.1, R76.1
- new net N$108: C68.1, IC14.OUT
- new net N$109: C72.1, IC15.+IN1, R81.1
- new net N$110: IC16.-IN, R79.1, R80.1
- new net N$111: IC16.OUT, R80.2, R84.2
- new net N$112: IC15.-IN1, R82.1, R83.1
- new net N$113: C73.1, R78.1, R81.2
- new net N$114: C73.2, IC15.OUT1, R79.2, R83.2
- new net N$115: C74.2, IC3.AIN3, R84.1
- new net N$116: IN5.2, R88.1
- new net N$117: IN5.4, R85.1
- new net N$118: IN5.1, R86.1
- new net N$119: IC17.-IN, R89.2
- new net N$120: C75.1, C76.1, D17.AC, R85.2, R89.1
- new net N$121: C75.2, C77.2, D18.AC, R86.2, R90.1
- new net N$122: IC17.-RG, IC18.+IN3, R91.2
- new net N$123: IC17.+RG, IC18.+IN4, R91.1
- new net N$124: IC17.+IN, R90.2
- new net N$125: D20.AC, IC18.-IN4, IC18.OUT4, R88.2, R93.1
- new net N$126: D19.AC, IC18.-IN3, IC18.OUT3, R87.2, R92.1
- new net N$127: C83.2, IC18.+IN2, R97.1
- new net N$128: IC18.-IN2, R94.2, R95.2
- new net N$129: C82.2, C83.1, R96.1
- new net N$130: C82.1, IC17.OUT
- new net N$131: C86.1, IC18.+IN1, R101.1
- new net N$132: IC19.-IN, R100.1, R99.1
- new net N$133: IC19.OUT, R100.2, R104.2
- new net N$134: IC18.-IN1, R102.1, R103.1
- new net N$135: C87.1, R101.2, R98.1
- new net N$136: C87.2, IC18.OUT1, R103.2, R99.2
- new net N$137: C88.2, IC3.AIN4, R104.1
- new net N$138: IN6.3, R107.1
- new net N$139: IN6.2, R108.1
- new net N$140: IN6.4, R105.1
- new net N$141: IN6.1, R106.1
- new net N$142: IC20.-IN, R109.2
- new net N$143: C89.1, C90.1, D21.AC, R105.2, R109.1
- new net N$144: C89.2, C91.2, D22.AC, R106.2, R110.1
- new net N$145: IC20.-RG, IC21.+IN3, R111.2
- new net N$146: IC20.+RG, IC21.+IN4, R111.1
- new net N$147: IC20.+IN, R110.2
- new net N$148: D24.AC, IC21.-IN4, IC21.OUT4, R108.2, R113.1
- new net N$149: D23.AC, IC21.-IN3, IC21.OUT3, R107.2, R112.1
- new net N$150: C97.2, IC21.+IN2, R117.1
- new net N$151: IC21.-IN2, R114.2, R115.2
- new net N$152: C96.2, C97.1, R116.1
- new net N$153: C96.1, IC20.OUT
- new net N$154: C100.1, IC21.+IN1, R121.1
- new net N$155: IC22.-IN, R119.1, R120.1
- new net N$156: IC22.OUT, R120.2, R124.2
- new net N$157: IC21.-IN1, R122.1, R123.1
- new net N$158: C101.1, R118.1, R121.2
- new net N$159: C101.2, IC21.OUT1, R119.2, R123.2
- new net N$160: C102.2, IC3.AIN5, R124.1
- new net N$161: IN7.3, R127.1
- new net N$162: IN7.2, R128.1
- new net N$163: IN7.4, R125.1
- new net N$164: IN7.1, R126.1
- new net N$165: IC23.-IN, R129.2
- new net N$166: C103.1, C104.1, D25.AC, R125.2, R129.1
- new net N$167: C103.2, C105.2, D26.AC, R126.2, R130.1
- new net N$168: IC23.-RG, IC24.+IN3, R131.2
- new net N$169: IC23.+RG, IC24.+IN4, R131.1
- new net N$170: IC23.+IN, R130.2
- new net N$171: D28.AC, IC24.-IN4, IC24.OUT4, R128.2, R133.1
- new net N$172: D27.AC, IC24.-IN3, IC24.OUT3, R127.2, R132.1
- new net N$173: C111.2, IC24.+IN2, R137.1
- new net N$174: IC24.-IN2, R134.2, R135.2
- new net N$175: C110.2, C111.1, R136.1
- new net N$176: C110.1, IC23.OUT
- new net N$177: C114.1, IC24.+IN1, R141.1
- new net N$178: IC25.-IN, R139.1, R140.1
- new net N$179: IC25.OUT, R140.2, R144.2
- new net N$180: IC24.-IN1, R142.1, R143.1
- new net N$181: C115.1, R138.1, R141.2
- new net N$182: C115.2, IC24.OUT1, R139.2, R143.2
- new net N$184: C130.2, IC3.AIN7, R164.1
- new net N$185: IN8.3, R147.1
- new net N$186: IN8.2, R148.1
- new net N$187: IN8.4, R145.1
- new net N$188: IN8.1, R146.1
- new net N$189: IC26.-IN, R149.2
- new net N$190: C117.1, C118.1, D29.AC, R145.2, R149.1
- new net N$191: C117.2, C119.2, D30.AC, R146.2, R150.1
- new net N$192: IC26.-RG, IC27.+IN3, R151.2
- new net N$193: IC26.+RG, IC27.+IN4, R151.1
- new net N$194: IC26.+IN, R150.2
- new net N$195: D32.AC, IC27.-IN4, IC27.OUT4, R148.2, R153.1
- new net N$196: D31.AC, IC27.-IN3, IC27.OUT3, R147.2, R152.1
- new net N$197: C125.2, IC27.+IN2, R157.1
- new net N$198: IC27.-IN2, R154.2, R155.2
- new net N$199: C124.2, C125.1, R156.1
- new net N$200: C124.1, IC26.OUT
- new net N$201: C128.1, IC27.+IN1, R161.1
- new net N$202: IC28.-IN, R159.1, R160.1
- new net N$203: IC28.OUT, R160.2, R164.2
- new net N$204: IC27.-IN1, R162.1, R163.1
- new net N$205: C129.1, R158.1, R161.2
- new net N$206: C129.2, IC27.OUT1, R159.2, R163.2
- new net N$39: C22.+, C24.1, G1.+VOUT, IC5.VI1, L1.2
- new net N$44: C23.-, C25.2, G1.-VOUT, L2.2
- new net N$45: IN2.2, R28.1
- new net N$46: IN2.4, R24.1
- new net N$47: IN2.1, R26.1
- new net N$48: IC8.-IN, R29.2
- new net N$49: C30.1, C31.1, D5.AC, R24.2, R29.1
- new net N$50: C30.2, C32.2, D6.AC, R26.2, R30.1
- new net N$51: IC8.-RG, IC9.+IN3, R31.2
- new net N$52: IC8.+RG, IC9.+IN4, R31.1
- new net N$53: IC8.+IN, R30.2
- new net N$54: D8.AC, IC9.-IN4, IC9.OUT4, R28.2, R33.1
- new net N$55: D7.AC, IC9.-IN3, IC9.OUT3, R27.2, R32.1
- new net N$56: C38.2, IC9.+IN2, R37.1
- new net N$57: IC9.-IN2, R34.2, R35.2
- new net N$58: C37.2, C38.1, R36.1
- new net N$59: C37.1, IC8.OUT
- new net N$60: C41.1, IC9.+IN1, R41.1
- new net N$61: IC10.-IN, R39.1, R40.1
- new net N$62: IC10.OUT, R40.2, R44.2
- new net N$63: C56.2, IC2.OUT1, R22.2, R23.2
- new net N$64: IC9.-IN1, R42.1, R43.1
- new net N$65: C42.1, R38.1, R41.2
- new net N$66: C42.2, IC9.OUT1, R39.2, R43.2
- new net N$67: C43.2, IC3.AIN1, R44.1
- new net N$68: IN3.3, R47.1
- new net N$69: IN3.2, R48.1
- new net N$70: IN3.4, R45.1
- new net N$71: IN3.1, R46.1
- new net N$72: IC11.-IN, R49.2
- new net N$73: C45.1, C46.1, D9.AC, R45.2, R49.1
- new net N$74: C45.2, C47.2, D10.AC, R46.2, R50.1
- new net N$75: IC11.-RG, IC12.+IN3, R51.2
- new net N$76: IC11.+RG, IC12.+IN4, R51.1
- new net N$77: IC11.+IN, R50.2
- new net N$78: D12.AC, IC12.-IN4, IC12.OUT4, R48.2, R53.1
- new net N$79: D11.AC, IC12.-IN3, IC12.OUT3, R47.2, R52.1
- new net N$80: C54.2, IC12.+IN2, R57.1
- new net N$81: IC12.-IN2, R54.2, R55.2
- new net N$82: C53.2, C54.1, R56.1
- new net N$83: C53.1, IC11.OUT
- new net N$84: C58.1, IC12.+IN1, R61.1
- new net N$85: IC13.-IN, R59.1, R60.1
- new net N$86: IC13.OUT, R60.2, R64.2
- new net N$87: IC12.-IN1, R62.1, R63.1
- new net N$88: C59.1, R58.1, R61.2
- new net N$89: C59.2, IC12.OUT1, R59.2, R63.2
- new net N$90: C60.2, IC3.AIN2, R64.1
- new net N$91: C116.2, IC3.AIN6, R144.1
- new net N$92: IN5.3, R87.1
- new net N$93: IN4.3, R67.1
- new net N$94: IN4.2, R68.1
- new net N$95: IN4.4, R65.1
- new net N$96: IN4.1, R66.1
- new net N$97: IC14.-IN, R69.2
- new net N$98: C61.1, C62.1, D13.AC, R65.2, R69.1
- new net N$99: C61.2, C63.2, D14.AC, R66.2, R70.1
- net +3.3V: now also C21.+, C44.1, IC5.VO; no longer IC5.VCC
- net +5VA: now also C107.2, C108.1, C112.1, C121.2, C122.1, C126.1, C26.1, C27.+, C34.2, C35.1, C39.1, C49.2, C50.1, C55.1, C65.2, C66.1, C70.1, C79.2, C80.1, C84.1, C93.2, C94.1, C98.1, D10.C, D11.C, D12.C, D13.C, D14.C, D15.C, D16.C, D17.C, D18.C, D19.C, D20.C, D21.C, D22.C, D23.C, D24.C, D25.C, D26.C, D27.C, D28.C, D29.C, D30.C, D31.C, D32.C, D5.C, D6.C, D7.C, D8.C, D9.C, IC10.+VS, IC11.+VS, IC12.+VS, IC13.+VS, IC14.+VS, IC15.+VS, IC16.+VS, IC17.+VS, IC18.+VS, IC19.+VS, IC20.+VS, IC21.+VS, IC22.+VS, IC23.+VS, IC24.+VS, IC25.+VS, IC26.+VS, IC27.+VS, IC28.+VS, IC7.VIN, IC8.+VS, IC9.+VS, L1.1
- net -5VA: now also C106.1, C109.2, C120.1, C123.2, C28.2, C29.-, C33.1, C36.2, C48.1, C51.2, C64.1, C67.2, C78.1, C81.2, C92.1, C95.2, D10.A, D11.A, D12.A, D13.A, D14.A, D15.A, D16.A, D17.A, D18.A, D19.A, D20.A, D21.A, D22.A, D23.A, D24.A, D25.A, D26.A, D27.A, D28.A, D29.A, D30.A, D31.A, D32.A, D5.A, D6.A, D7.A, D8.A, D9.A, IC11.-VS, IC12.-VS, IC14.-VS, IC15.-VS, IC17.-VS, IC18.-VS, IC20.-VS, IC21.-VS, IC23.-VS, IC24.-VS, IC26.-VS, IC27.-VS, IC8.-VS, IC9.-VS, L2.1
- net CH1SW1: now also R20.2; no longer IC5.NC1, R19.2
- net CH1SW2: now also IC9.OUT2, R35.1, R36.2, R38.2; no longer IC5.COM1, R19.1, R20.2
- net GND: now also C100.2, C102.1, C104.2, C105.1, C106.2, C107.1, C108.2, C109.1, C112.2, C113.1, C114.2, C116.1, C118.2, C119.1, C120.2, C121.1, C122.2, C123.1, C126.2, C127.1, C128.2, C130.1, C14.2, C19.1, C20.-, C21.-, C22.-, C23.+, C24.2, C25.1, C26.2, C27.-, C28.1, C29.+, C31.2, C32.1, C33.2, C34.1, C35.2, C36.1, C39.2, C40.1, C41.2, C43.1, C44.2, C46.2, C47.1, C48.2, C49.1, C50.2, C51.1, C52.1, C55.2, C57.1, C58.2, C60.1, C62.2, C63.1, C64.2, C65.1, C66.2, C67.1, C70.2, C71.1, C72.2, C74.1, C76.2, C77.1, C78.2, C79.1, C80.2, C81.1, C84.2, C85.1, C86.2, C88.1, C90.2, C91.1, C92.2, C93.1, C94.2, C95.1, C98.2, C99.1, G1.COM, IC10.-VS, IC11.REF, IC13.-VS, IC14.REF, IC16.-VS, IC17.REF, IC19.-VS, IC20.REF, IC22.-VS, IC23.REF, IC25.-VS, IC26.REF, IC28.-VS, IC7.GND, IC8.REF, R102.2, R112.2, R113.2, R114.1, R117.2, R122.2, R132.2, R133.2, R134.1, R137.2, R142.2, R152.2, R153.2, R154.1, R157.2, R162.2, R21.2, R32.2, R33.2, R34.1, R37.2, R42.2, R52.2, R53.2, R54.1, R57.2, R62.2, R72.2, R73.2, R74.1, R77.2, R82.2, R92.2, R93.2, R94.1, R97.2; no longer DC1.COM, R18.1, R23.2
- net N$19: now also IC2.-IN1, R21.1; no longer IC4.+IN, R24.2
- net N$20: now also C14.1, R19.1; no longer R18.2
- net N$21: now also R18.2; no longer IC3.AIN0
- net N$28: now also C19.2, IC3.AIN0, R18.1; no longer C14.2, IC2.OUT1, R21.1, R22.2
- net N$29: now also C56.1, R19.2; no longer C14.1, IC2.-IN1, R21.2
- net N$31: now also IN2.3, R27.1; no longer IC3.D0/CLKOUT, IC5.IN1, IC5.IN2
- net N$36: now also G1.+VIN; no longer DC1.+VIN
- net N$37: now also G1.-VIN; no longer DC1.-VIN
- net VREF: now also C113.2, C127.2, C20.+, C40.2, C52.2, C57.2, C71.2, C85.2, C99.2, IC10.+IN, IC13.+IN, IC16.+IN, IC19.+IN, IC22.+IN, IC25.+IN, IC28.+IN, IC3.AINCOM, IC4.+IN, IC7.VOUT; no longer R24.1
Other:
- moved on the sheet: C12, C13, C14, R10, R11, R12, R13, R18, R19, R20, R21, R23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

Commit message: Latest modification for all-in-one board
Connections:
- new net N$207: G1.-VIN, INT.2
- net N$37: no longer G1.-VIN, INT.3
- net N$38: now also INT.3; no longer INT.2
Changed lines of the file:
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@@
 <net name="N$37" class="0">
 <segment>
-<wire x1="695.96" y1="-167.64" x2="695.96" y2="-2.54" width="0.1524" layer="91"/>
 <pinref part="IC6" gate="G$1" pin="GND2_"/>
 <wire x1="695.96" y1="-2.54" x2="690.88" y2="-2.54" width="0.1524" layer="91"/>
@@
 <wire x1="695.96" y1="58.42" x2="698.5" y2="58.42" width="0.1524" layer="91"/>
 <junction x="695.96" y="58.42"/>
-<pinref part="INT" gate="A" pin="3"/>
-<wire x1="772.16" y1="22.86" x2="762" y2="22.86" width="0.1524" layer="91"/>
-<wire x1="762" y1="22.86" x2="762" y2="10.16" width="0.1524" layer="91"/>
 <pinref part="INT" gate="A" pin="8"/>
 <wire x1="762" y1="10.16" x2="772.16" y2="10.16" width="0.1524" layer="91"/>
 <wire x1="695.96" y1="-2.54" x2="762" y2="-2.54" width="0.1524" layer="91"/>
 <wire x1="762" y1="-2.54" x2="762" y2="10.16" width="0.1524" layer="91"/>
-<junction x="762" y="10.16"/>
-<pinref part="G1" gate="G$1" pin="-VIN"/>
-<wire x1="657.86" y1="-167.64" x2="695.96" y2="-167.64" width="0.1524" layer="91"/>
 </segment>
 </net>
@@
 <pinref part="IC6" gate="G$1" pin="VE2"/>
 <wire x1="690.88" y1="7.62" x2="708.66" y2="7.62" width="0.1524" layer="91"/>
-<wire x1="708.66" y1="7.62" x2="708.66" y2="25.4" width="0.1524" layer="91"/>
 <pinref part="IC6" gate="G$1" pin="VDD2"/>
-<wire x1="708.66" y1="25.4" x2="708.66" y2="58.42" width="0.1524" layer="91"/>
+<wire x1="708.66" y1="7.62" x2="708.66" y2="22.86" width="0.1524" layer="91"/>
+<wire x1="708.66" y1="22.86" x2="708.66" y2="58.42" width="0.1524" layer="91"/>
 <wire x1="708.66" y1="58.42" x2="708.66" y2="68.58" width="0.1524" layer="91"/>
 <wire x1="708.66" y1="68.58" x2="690.88" y2="68.58" width="0.1524" layer="91"/>
@@
 <wire x1="706.12" y1="58.42" x2="708.66" y2="58.42" width="0.1524" layer="91"/>
 <junction x="708.66" y="58.42"/>
-<pinref part="INT" gate="A" pin="2"/>
-<wire x1="772.16" y1="25.4" x2="708.66" y2="25.4" width="0.1524" layer="91"/>
-<junction x="708.66" y="25.4"/>
+<pinref part="INT" gate="A" pin="3"/>
+<wire x1="772.16" y1="22.86" x2="708.66" y2="22.86" width="0.1524" layer="91"/>
+<junction x="708.66" y="22.86"/>
 </segment>
 </net>
@@
 </segment>
 </net>
+<net name="N$207" class="0">
+<segment>
+<pinref part="G1" gate="G$1" pin="-VIN"/>
+<wire x1="657.86" y1="-167.64" x2="789.94" y2="-167.64" width="0.1524" layer="91"/>
+<wire x1="789.94" y1="-167.64" x2="789.94" y2="40.64" width="0.1524" layer="91"/>
+<wire x1="789.94" y1="40.64" x2="759.46" y2="40.64" width="0.1524" layer="91"/>
+<wire x1="759.46" y1="40.64" x2="759.46" y2="25.4" width="0.1524" layer="91"/>
+<pinref part="INT" gate="A" pin="2"/>
+<wire x1="759.46" y1="25.4" x2="772.16" y2="25.4" width="0.1524" layer="91"/>
+</segment>
+</net>
