File: AllInOne.brd (EAGLE design)
At the start: 132.1 x 64.1 mm, 368 parts, among them IC1 AD8221ARZ, IC10 AD8605ARTZ, IC11 AD8221ARZ, IC12 TLC2254ID, IC13 AD8605ARTZ, IC14 AD8221ARZ, IC15 TLC2254ID, IC16 AD8605ARTZ, IC17 AD8221ARZ, IC18 TLC2254ID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

Commit message: Rename lbr
Parts:
- G1: device nanoeeg:TMV0505D -> femtoexg:TMV0505D
- IC1, IC11, IC14, IC17, IC20, IC23, IC26, IC8: device nanoeeg:SO-08 -> femtoexg:SO-08
- IC10, IC13, IC16, IC19, IC22, IC25, IC28, IC4: device nanoeeg:AD8605ARTZ -> femtoexg:AD8605ARTZ
- IC12, IC15, IC18, IC2, IC21, IC24, IC27, IC9: device nanoeeg:TLC2254ID -> femtoexg:TLC2254ID
- IC3: device nanoeeg:ADS1256IDBT -> femtoexg:ADS1256IDBT
- IC6: device nanoeeg:ADUM1402ARWZ -> femtoexg:ADUM1402ARWZ
- IC7: device nanoeeg:REF3125AIDBZT -> femtoexg:REF3125AIDBZT
