File: AllInOne.sch (EAGLE design)
At the start: 368 parts, among them IC1 AD8221ARZ, IC10 AD8605ARTZ, IC11 AD8221ARZ, IC12 TLC2254ID, IC13 AD8605ARTZ, IC14 AD8221ARZ, IC15 TLC2254ID, IC16 AD8605ARTZ, IC17 AD8221ARZ, IC18 TLC2254ID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

Commit message: Rename lbr
Parts:
- G1: device nanoeeg:TMV0505D -> femtoexg:TMV0505D
- IC1, IC11, IC14, IC17, IC20, IC23, IC26, IC8: device nanoeeg:AD8221ARZ -> femtoexg:AD8221ARZ
- IC10, IC13, IC16, IC19, IC22, IC25, IC28, IC4: device nanoeeg:AD8605ARTZ -> femtoexg:AD8605ARTZ
- IC12, IC15, IC18, IC2, IC21, IC24, IC27, IC9: device nanoeeg:TLC2254ID -> femtoexg:TLC2254ID
- IC3: device nanoeeg:ADS1256IDBT -> femtoexg:ADS1256IDBT
- IC6: device nanoeeg:ADUM1402ARWZ -> femtoexg:ADUM1402ARWZ
- IC7: device nanoeeg:REF3125AIDBZT -> femtoexg:REF3125AIDBZT
Changed lines of the file:
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@@
 <part name="C2" library="rcl" deviceset="C-EU" device="C0805" value="100pF"/>
 <part name="C3" library="rcl" deviceset="C-EU" device="C0805" value="100pF"/>
-<part name="IC1" library="nanoeeg" deviceset="AD8221ARZ" device=""/>
+<part name="IC1" library="femtoexg" deviceset="AD8221ARZ" device=""/>
 <part name="R7" library="rcl" deviceset="R-EU_" device="R0805" value="2K"/>
 <part name="C4" library="rcl" deviceset="C-EU" device="C0805" value="0.1"/>
@@
 <part name="COM" library="pinhead" deviceset="PINHD-1X2" device="" value="COM"/>
 <part name="GND16" library="supply1" deviceset="GND" device=""/>
-<part name="IC2" library="nanoeeg" deviceset="TLC2254ID" device=""/>
-<part name="IC3" library="nanoeeg" deviceset="ADS1256IDBT" device=""/>
-<part name="IC4" library="nanoeeg" deviceset="AD8605ARTZ" device=""/>
+<part name="IC2" library="femtoexg" deviceset="TLC2254ID" device=""/>
+<part name="IC3" library="femtoexg" deviceset="ADS1256IDBT" device=""/>
+<part name="IC4" library="femtoexg" deviceset="AD8605ARTZ" device=""/>
 <part name="GND17" library="supply1" deviceset="GND" device=""/>
 <part name="R20" library="rcl" deviceset="R-EU_" device="R0805" value="100K"/>
@@
 <part name="C16" library="rcl" deviceset="C-EU" device="C0805" value="0.1"/>
 <part name="GND22" library="supply1" deviceset="GND" device=""/>
-<part name="IC6" library="nanoeeg" deviceset="ADUM1402ARWZ" device=""/>
+<part name="IC6" library="femtoexg" deviceset="ADUM1402ARWZ" device=""/>
 <part name="GND23" library="supply1" deviceset="GND" device=""/>
 <part name="GND24" library="supply1" deviceset="GND" device=""/>
@@
 <part name="C19" library="rcl" deviceset="C-EU" device="C0805" value="0.1"/>
 <part name="GND21" library="supply1" deviceset="GND" device=""/>
-<part name="G1" library="nanoeeg" deviceset="TMV0505D" device=""/>
+<part name="G1" library="femtoexg" deviceset="TMV0505D" device=""/>
 <part name="IC5" library="linear" deviceset="MCP1703*" device="MB" technology="33"/>
 <part name="GND27" library="supply1" deviceset="GND" device=""/>
-<part name="IC7" library="nanoeeg" deviceset="REF3125AIDBZT" device=""/>
+<part name="IC7" library="femtoexg" deviceset="REF3125AIDBZT" device=""/>
 <part name="GND28" library="supply1" deviceset="GND" device=""/>
 <part name="C20" library="rcl" deviceset="CPOL-EU" device="E2-4" value="47u"/>
@@
 <part name="C31" library="rcl" deviceset="C-EU" device="C0805" value="100pF"/>
 <part name="C32" library="rcl" deviceset="C-EU" device="C0805" value="100pF"/>
-<part name="IC8" library="nanoeeg" deviceset="AD8221ARZ" device=""/>
+<part name="IC8" library="femtoexg" deviceset="AD8221ARZ" device=""/>
 <part name="R31" library="rcl" deviceset="R-EU_" device="R0805" value="2K"/>
 <part name="C33" library="rcl" deviceset="C-EU" device="C0805" value="0.1"/>
@@
 <part name="R37" library="rcl" deviceset="R-EU_" device="R0805" value="100K"/>
 <part name="GND39" library="supply1" deviceset="GND" device=""/>
-<part name="IC9" library="nanoeeg" deviceset="TLC2254ID" device=""/>
-<part name="IC10" library="nanoeeg" deviceset="AD8605ARTZ" device=""/>
+<part name="IC9" library="femtoexg" deviceset="TLC2254ID" device=""/>
+<part name="IC10" library="femtoexg" deviceset="AD8605ARTZ" device=""/>
 <part name="GND40" library="supply1" deviceset="GND" device=""/>
 <part name="R38" library="rcl" deviceset="R-EU_" device="R0805" value="100K"/>
@@
 <part name="C46" library="rcl" deviceset="C-EU" device="C0805" value="100pF"/>
 <part name="C47" library="rcl" deviceset="C-EU" device="C0805" value="100pF"/>
-<part name="IC11" library="nanoeeg" deviceset="AD8221ARZ" device=""/>
+<part name="IC11" library="femtoexg" deviceset="AD8221ARZ" device=""/>
 <part name="R51" library="rcl" deviceset="R-EU_" device="R0805" value="2K"/>
 <part name="C48" library="rcl" deviceset="C-EU" device="C0805" value="0.1"/>
@@
 <part name="R57" library="rcl" deviceset="R-EU_" device="R0805" value="100K"/>
 <part name="GND56" library="supply1" deviceset="GND" device=""/>
-<part name="IC12" library="nanoeeg" deviceset="TLC2254ID" device=""/>
-<part name="IC13" library="nanoeeg" deviceset="AD8605ARTZ" device=""/>
+<part name="IC12" library="femtoexg" deviceset="TLC2254ID" device=""/>
+<part name="IC13" library="femtoexg" deviceset="AD8605ARTZ" device=""/>
 <part name="GND57" library="supply1" deviceset="GND" device=""/>
 <part name="R58" library="rcl" deviceset="R-EU_" device="R0805" value="100K"/>
@@
 <part name="C62" library="rcl" deviceset="C-EU" device="C0805" value="100pF"/>
 <part name="C63" library="rcl" deviceset="C-EU" device="C0805" value="100pF"/>
-<part name="IC14" library="nanoeeg" deviceset="AD8221ARZ" device=""/>
+<part name="IC14" library="femtoexg" deviceset="AD8221ARZ" device=""/>
 <part name="R71" library="rcl" deviceset="R-EU_" device="R0805" value="2K"/>
 <part name="C64" library="rcl" deviceset="C-EU" device="C0805" value="0.1"/>
@@
 <part name="R77" library="rcl" deviceset="R-EU_" device="R0805" value="100K"/>
 <part name="GND73" library="supply1" deviceset="GND" device=""/>
-<part name="IC15" library="nanoeeg" deviceset="TLC2254ID" device=""/>
-<part name="IC16" library="nanoeeg" deviceset="AD8605ARTZ" device=""/>
+<part name="IC15" library="femtoexg" deviceset="TLC2254ID" device=""/>
+<part name="IC16" library="femtoexg" deviceset="AD8605ARTZ" device=""/>
 <part name="GND74" library="supply1" deviceset="GND" device=""/>
 <part name="R78" library="rcl" deviceset="R-EU_" device="R0805" value="100K"/>
@@
 <part name="C76" library="rcl" deviceset="C-EU" device="C0805" value="100pF"/>
 <part name="C77" library="rcl" deviceset="C-EU" device="C0805" value="100pF"/>
-<part name="IC17" library="nanoeeg" deviceset="AD8221ARZ" device=""/>
+<part name="IC17" library="femtoexg" deviceset="AD8221ARZ" device=""/>
 <part name="R91" library="rcl" deviceset="R-EU_" device="R0805" value="2K"/>
 <part name="C78" library="rcl" deviceset="C-EU" device="C0805" value="0.1"/>
@@
 <part name="R97" library="rcl" deviceset="R-EU_" device="R0805" value="100K"/>
 <part name="GND89" library="supply1" deviceset="GND" device=""/>
-<part name="IC18" library="nanoeeg" deviceset="TLC2254ID" device=""/>
-<part name="IC19" library="nanoeeg" deviceset="AD8605ARTZ" device=""/>
+<part name="IC18" library="femtoexg" deviceset="TLC2254ID" device=""/>
+<part name="IC19" library="femtoexg" deviceset="AD8605ARTZ" device=""/>
 <part name="GND90" library="supply1" deviceset="GND" device=""/>
 <part name="R98" library="rcl" deviceset="R-EU_" device="R0805" value="100K"/>
@@
 <part name="C90" library="rcl" deviceset="C-EU" device="C0805" value="100pF"/>
 <part name="C91" library="rcl" deviceset="C-EU" device="C0805" value="100pF"/>
-<part name="IC20" library="nanoeeg" deviceset="AD8221ARZ" device=""/>
+<part name="IC20" library="femtoexg" deviceset="AD8221ARZ" device=""/>
 <part name="R111" library="rcl" deviceset="R-EU_" device="R0805" value="2K"/>
 <part name="C92" library="rcl" deviceset="C-EU" device="C0805" value="0.1"/>
@@
 <part name="R117" library="rcl" deviceset="R-EU_" device="R0805" value="100K"/>
 <part name="GND105" library="supply1" deviceset="GND" device=""/>
-<part name="IC21" library="nanoeeg" deviceset="TLC2254ID" device=""/>
-<part name="IC22" library="nanoeeg" deviceset="AD8605ARTZ" device=""/>
+<part name="IC21" library="femtoexg" deviceset="TLC2254ID" device=""/>
+<part name="IC22" library="femtoexg" deviceset="AD8605ARTZ" device=""/>
 <part name="GND106" library="supply1" deviceset="GND" device=""/>
 <part name="R118" library="rcl" deviceset="R-EU_" device="R0805" value="100K"/>
@@
 <part name="C104" library="rcl" deviceset="C-EU" device="C0805" value="100pF"/>
 <part name="C105" library="rcl" deviceset="C-EU" device="C0805" value="100pF"/>
-<part name="IC23" library="nanoeeg" deviceset="AD8221ARZ" device=""/>
+<part name="IC23" library="femtoexg" deviceset="AD8221ARZ" device=""/>
 <part name="R131" library="rcl" deviceset="R-EU_" device="R0805" value="2K"/>
 <part name="C106" library="rcl" deviceset="C-EU" device="C0805" value="0.1"/>
@@
 <part name="R137" library="rcl" deviceset="R-EU_" device="R0805" value="100K"/>
 <part name="GND121" library="supply1" deviceset="GND" device=""/>
-<part name="IC24" library="nanoeeg" deviceset="TLC2254ID" device=""/>
-<part name="IC25" library="nanoeeg" deviceset="AD8605ARTZ" device=""/>
+<part name="IC24" library="femtoexg" deviceset="TLC2254ID" device=""/>
+<part name="IC25" library="femtoexg" deviceset="AD8605ARTZ" device=""/>
 <part name="GND122" library="supply1" deviceset="GND" device=""/>
 <part name="R138" library="rcl" deviceset="R-EU_" device="R0805" value="100K"/>
@@
 <part name="C118" library="rcl" deviceset="C-EU" device="C0805" value="100pF"/>
 <part name="C119" library="rcl" deviceset="C-EU" device="C0805" value="100pF"/>
-<part name="IC26" library="nanoeeg" deviceset="AD8221ARZ" device=""/>
+<part name="IC26" library="femtoexg" deviceset="AD8221ARZ" device=""/>
 <part name="R151" library="rcl" deviceset="R-EU_" device="R0805" value="2K"/>
 <part name="C120" library="rcl" deviceset="C-EU" device="C0805" value="0.1"/>
@@
 <part name="R157" library="rcl" deviceset="R-EU_" device="R0805" value="100K"/>
 <part name="GND137" library="supply1" deviceset="GND" device=""/>
-<part name="IC27" library="nanoeeg" deviceset="TLC2254ID" device=""/>
-<part name="IC28" library="nanoeeg" deviceset="AD8605ARTZ" device=""/>
+<part name="IC27" library="femtoexg" deviceset="TLC2254ID" device=""/>
+<part name="IC28" library="femtoexg" deviceset="AD8605ARTZ" device=""/>
 <part name="GND138" library="supply1" deviceset="GND" device=""/>
 <part name="R158" library="rcl" deviceset="R-EU_" device="R0805" value="100K"/>
