File: Adc.sch (EAGLE design)
At the start: 4 parts, among them IC1 ADS1256IDBT, IC2 ADUM1402ARWZ, IC3 AD8605ARTZ

Commit message: .
Parts:
- added C1, C10, C11, C12, C13, C14, C15, C16, C17, C18, C19, C2, C20, C21, C22, C23, C24, C25, C26, C27, C3, C31, C32, C36, C37, C38, C4, C41, C42, C5, C6, C7, C8, C9: 0.1uF, rcl:C-EUC0805
- added C28, C33, C34, C35, C39, C40: 47uF, rcl:CPOL-EUE2-4
- added C29, C30: 18pF, rcl:C-EUC0805
- added IC10, IC4, IC5, IC6, IC7, IC8, IC9: AD8605ARTZ, nanoeeg:AD8605ARTZ
- added IC11: REF3125AIDBZT, nanoeeg:REF3125AIDBZT
- added IC12: MCP170333MB, linear:MCP170333MB
- added JP1, JP2, JP3, JP4, JP5, JP6, JP7, JP8: (no value), pinhead:PINHD-1X4
- added JP10: (no value), pinhead:PINHD-1X2
- added JP9: (no value), pinhead:PINHD-1X8
- added L1, L2, L3: (no value), rcl:L-USL4532P
- added Q1: 8MHz, crystal:CRYSTALHC49U-V
- added R1, R10, R13, R16, R19, R22, R25, R26, R27, R28, R4, R7: 100, rcl:R-EU_R0805
- added R11, R12, R14, R15, R17, R18, R2, R20, R21, R23, R24, R3, R5, R6, R8, R9: 1k, rcl:R-EU_R0805
Connections:
- new net +3.3V: C27.1, C35.+, C36.1, C41.2, IC1.DVDD, IC1.RESET, IC1.SYNC/PDWN, IC12.VO, IC2.VDD1, IC2.VE1
- new net +5VA: C11.1, C14.1, C17.1, C2.1, C20.1, C23.1, C25.2, C37.1, C39.+, C5.1, C8.1, IC1.AVDD, IC10.+VS, IC11.VIN, IC3.+VS, IC4.+VS, IC5.+VS, IC6.+VS, IC7.+VS, IC8.+VS, IC9.+VS, JP1.3, JP2.3, JP3.3, JP4.3, JP5.3, JP6.3, JP7.3, JP8.3, L1.1
- new net -5VA: C38.2, C40.-, JP1.4, JP2.4, JP3.4, JP4.4, JP5.4, JP6.4, JP7.4, JP8.4, L2.1
- new net GND: C1.1, C10.1, C11.2, C12.2, C13.1, C14.2, C15.2, C16.1, C17.2, C18.2, C19.1, C2.2, C20.2, C21.2, C22.1, C23.2, C24.2, C25.1, C26.2, C28.-, C3.2, C37.2, C38.1, C39.-, C4.1, C40.+, C5.2, C6.2, C7.1, C8.2, C9.2, IC1.AGND, IC1.VREFN, IC10.-VS, IC11.GND, IC3.-VS, IC4.-VS, IC5.-VS, IC6.-VS, IC7.-VS, IC8.-VS, IC9.-VS, JP1.2, JP10.1, JP10.2, JP2.2, JP3.2, JP4.2, JP5.2, JP6.2, JP7.2, JP8.2, L3.1
- new net GNDIO: C27.2, C29.2, C30.2, C31.2, C32.1, C33.-, C34.+, C35.-, C36.2, C41.1, G1.COM, IC1.CS, IC1.DGND, IC12.GND, IC2.GND1, IC2.GND1_, L3.2
- new net N$1: IC3.-IN, R2.2, R3.2
- new net N$10: IC5.OUT, R7.1, R9.1
- new net N$11: C9.1, IC1.AIN2, R7.2
- new net N$12: JP3.1, R8.1
- new net N$13: IC6.-IN, R11.2, R12.2
- new net N$14: IC6.OUT, R10.1, R12.1
- new net N$15: C12.1, IC1.AIN3, R10.2
- new net N$16: JP4.1, R11.1
- new net N$17: IC7.-IN, R14.2, R15.2
- new net N$18: IC7.OUT, R13.1, R15.1
- new net N$19: C15.1, IC1.AIN4, R13.2
- new net N$2: IC3.OUT, R1.1, R3.1
- new net N$20: JP5.1, R14.1
- new net N$21: IC8.-IN, R17.2, R18.2
- new net N$22: IC8.OUT, R16.1, R18.1
- new net N$23: C18.1, IC1.AIN5, R16.2
- new net N$24: JP6.1, R17.1
- new net N$25: IC9.-IN, R20.2, R21.2
- new net N$26: IC9.OUT, R19.1, R21.1
- new net N$27: C21.1, IC1.AIN6, R19.2
- new net N$28: JP7.1, R20.1
- new net N$29: IC10.-IN, R23.2, R24.2
- new net N$3: JP1.1, R2.1
- new net N$30: IC10.OUT, R22.1, R24.1
- new net N$31: C24.1, IC1.AIN7, R22.2
- new net N$32: JP8.1, R23.1
- new net N$33: C29.1, IC1.XTAL2, Q1.1
- new net N$34: C30.1, IC1.XTAL1/CLKIN, Q1.2
- new net N$35: IC2.VID, JP9.7
- new net N$36: IC1.DRDY, R25.1
- new net N$37: IC1.SCLK, R26.1
- new net N$38: IC1.DIN, R27.1
- new net N$39: IC1.DOUT, R28.1
- new net N$4: C3.1, IC1.AIN0, R1.2
- new net N$40: C42.1, IC2.GND2, IC2.GND2_, JP9.8
- new net N$41: C31.1, C33.+, G1.+VOUT, IC12.VI1, L1.2
- new net N$42: C32.2, C34.-, G1.-VOUT, L2.2
- new net N$43: C42.2, IC2.VDD2, IC2.VE2, JP9.3
- new net N$44: IC2.VIA, R25.2
- new net N$45: IC2.VIB, R28.2
- new net N$46: IC2.VOC, R26.2
- new net N$47: IC2.VOD, R27.2
- new net N$48: IC2.VIC, JP9.6
- new net N$49: IC2.VOB, JP9.5
- new net N$5: IC4.-IN, R5.2, R6.2
- new net N$50: IC2.VOA, JP9.4
- new net N$51: G1.+VIN, JP9.1
- new net N$52: G1.-VIN, JP9.2
- new net N$6: IC4.OUT, R4.1, R6.1
- new net N$7: C6.1, IC1.AIN1, R4.2
- new net N$8: JP2.1, R5.1
- new net N$9: IC5.-IN, R8.2, R9.2
- new net REF: C1.2, C10.2, C13.2, C16.2, C19.2, C22.2, C26.1, C28.+, C4.2, C7.2, IC1.AINCOM, IC1.VREFP, IC10.+IN, IC11.VOUT, IC3.+IN, IC4.+IN, IC5.+IN, IC6.+IN, IC7.+IN, IC8.+IN, IC9.+IN
Other:
- moved on the sheet: IC2, IC3

Commit message: Rename lbr
Parts:
- G1: device nanoeeg:TMV0505D -> femtoexg:TMV0505D
- IC1: device nanoeeg:ADS1256IDBT -> femtoexg:ADS1256IDBT
- IC10, IC3, IC4, IC5, IC6, IC7, IC8, IC9: device nanoeeg:AD8605ARTZ -> femtoexg:AD8605ARTZ
- IC11: device nanoeeg:REF3125AIDBZT -> femtoexg:REF3125AIDBZT
- IC2: device nanoeeg:ADUM1402ARWZ -> femtoexg:ADUM1402ARWZ
Changed lines of the file:
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@@
 </classes>
 <parts>
-<part name="IC1" library="nanoeeg" deviceset="ADS1256IDBT" device=""/>
-<part name="IC2" library="nanoeeg" deviceset="ADUM1402ARWZ" device=""/>
-<part name="G1" library="nanoeeg" deviceset="TMV0505D" device=""/>
-<part name="IC3" library="nanoeeg" deviceset="AD8605ARTZ" device=""/>
+<part name="IC1" library="femtoexg" deviceset="ADS1256IDBT" device=""/>
+<part name="IC2" library="femtoexg" deviceset="ADUM1402ARWZ" device=""/>
+<part name="G1" library="femtoexg" deviceset="TMV0505D" device=""/>
+<part name="IC3" library="femtoexg" deviceset="AD8605ARTZ" device=""/>
 <part name="C1" library="rcl" deviceset="C-EU" device="C0805" value="0.1uF"/>
 <part name="GND1" library="supply1" deviceset="GND" device=""/>
@@
 <part name="JP1" library="pinhead" deviceset="PINHD-1X4" device=""/>
 <part name="GND5" library="supply1" deviceset="GND" device=""/>
-<part name="IC4" library="nanoeeg" deviceset="AD8605ARTZ" device=""/>
+<part name="IC4" library="femtoexg" deviceset="AD8605ARTZ" device=""/>
 <part name="C4" library="rcl" deviceset="C-EU" device="C0805" value="0.1uF"/>
 <part name="GND6" library="supply1" deviceset="GND" device=""/>
@@
 <part name="JP2" library="pinhead" deviceset="PINHD-1X4" device=""/>
 <part name="GND10" library="supply1" deviceset="GND" device=""/>
-<part name="IC5" library="nanoeeg" deviceset="AD8605ARTZ" device=""/>
+<part name="IC5" library="femtoexg" deviceset="AD8605ARTZ" device=""/>
 <part name="C7" library="rcl" deviceset="C-EU" device="C0805" value="0.1uF"/>
 <part name="GND11" library="supply1" deviceset="GND" device=""/>
@@
 <part name="JP3" library="pinhead" deviceset="PINHD-1X4" device=""/>
 <part name="GND15" library="supply1" deviceset="GND" device=""/>
-<part name="IC6" library="nanoeeg" deviceset="AD8605ARTZ" device=""/>
+<part name="IC6" library="femtoexg" deviceset="AD8605ARTZ" device=""/>
 <part name="C10" library="rcl" deviceset="C-EU" device="C0805" value="0.1uF"/>
 <part name="GND16" library="supply1" deviceset="GND" device=""/>
@@
 <part name="JP4" library="pinhead" deviceset="PINHD-1X4" device=""/>
 <part name="GND20" library="supply1" deviceset="GND" device=""/>
-<part name="IC7" library="nanoeeg" deviceset="AD8605ARTZ" device=""/>
+<part name="IC7" library="femtoexg" deviceset="AD8605ARTZ" device=""/>
 <part name="C13" library="rcl" deviceset="C-EU" device="C0805" value="0.1uF"/>
 <part name="GND21" library="supply1" deviceset="GND" device=""/>
@@
 <part name="JP5" library="pinhead" deviceset="PINHD-1X4" device=""/>
 <part name="GND25" library="supply1" deviceset="GND" device=""/>
-<part name="IC8" library="nanoeeg" deviceset="AD8605ARTZ" device=""/>
+<part name="IC8" library="femtoexg" deviceset="AD8605ARTZ" device=""/>
 <part name="C16" library="rcl" deviceset="C-EU" device="C0805" value="0.1uF"/>
 <part name="GND26" library="supply1" deviceset="GND" device=""/>
@@
 <part name="JP6" library="pinhead" deviceset="PINHD-1X4" device=""/>
 <part name="GND30" library="supply1" deviceset="GND" device=""/>
-<part name="IC9" library="nanoeeg" deviceset="AD8605ARTZ" device=""/>
+<part name="IC9" library="femtoexg" deviceset="AD8605ARTZ" device=""/>
 <part name="C19" library="rcl" deviceset="C-EU" device="C0805" value="0.1uF"/>
 <part name="GND31" library="supply1" deviceset="GND" device=""/>
@@
 <part name="JP7" library="pinhead" deviceset="PINHD-1X4" device=""/>
 <part name="GND35" library="supply1" deviceset="GND" device=""/>
-<part name="IC10" library="nanoeeg" deviceset="AD8605ARTZ" device=""/>
+<part name="IC10" library="femtoexg" deviceset="AD8605ARTZ" device=""/>
 <part name="C22" library="rcl" deviceset="C-EU" device="C0805" value="0.1uF"/>
 <part name="GND36" library="supply1" deviceset="GND" device=""/>
@@
 <part name="C28" library="rcl" deviceset="CPOL-EU" device="E2-4" value="47uF"/>
 <part name="GND43" library="supply1" deviceset="GND" device=""/>
-<part name="IC11" library="nanoeeg" deviceset="REF3125AIDBZT" device=""/>
+<part name="IC11" library="femtoexg" deviceset="REF3125AIDBZT" device=""/>
 <part name="GND44" library="supply1" deviceset="GND" device=""/>
 <part name="Q1" library="crystal" deviceset="CRYSTAL" device="HC49U-V" value="8MHz"/>

Commit message: Dimensions
Parts:
- removed L3: (no value), rcl:L-USL4532P
- added C43: 100pF, rcl:C-EUC0805
Connections:
- removed net GNDIO: C27.2, C29.2, C30.2, C31.2, C32.1, C33.-, C34.+, C35.-, C36.2, C41.1, G1.COM, IC1.CS, IC1.DGND, IC12.GND, IC2.GND1, IC2.GND1_, L3.2
- net GND: now also C27.2, C29.2, C30.2, C31.2, C32.1, C33.-, C34.+, C35.-, C36.2, C41.1, C43.2, G1.COM, IC1.CS, IC1.DGND, IC12.GND, IC2.GND1, IC2.GND1_; no longer L3.1
- net N$51: now also JP9.2; no longer JP9.1
- net N$52: now also JP9.1; no longer JP9.2
- net REF: now also C43.1
Other:
- moved on the sheet: C26, C28

Commit message: Routing
Parts:
- added JP11: (no value), pinhead:PINHD-1X2
- JP10: device pinhead:PINHD-1X2 -> pinhead:PINHD-1X1
- Q1: value 8MHz -> 7.68MHz
Connections:
- net GND: no longer JP10.2
- net N$51: now also JP11.1; no longer JP9.2
- net N$52: now also JP11.2; no longer JP9.1
Changed lines of the file:
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@@
 <part name="IC11" library="femtoexg" deviceset="REF3125AIDBZT" device=""/>
 <part name="GND44" library="supply1" deviceset="GND" device=""/>
-<part name="Q1" library="crystal" deviceset="CRYSTAL" device="HC49U-V" value="8MHz"/>
+<part name="Q1" library="crystal" deviceset="CRYSTAL" device="HC49U-V" value="7.68MHz"/>
 <part name="C29" library="rcl" deviceset="C-EU" device="C0805" value="18pF"/>
 <part name="C30" library="rcl" deviceset="C-EU" device="C0805" value="18pF"/>
@@
 <part name="JP9" library="pinhead" deviceset="PINHD-1X8" device=""/>
 <part name="C42" library="rcl" deviceset="C-EU" device="C0805" value="0.1uF"/>
-<part name="JP10" library="pinhead" deviceset="PINHD-1X2" device=""/>
 <part name="GND53" library="supply1" deviceset="GND" device=""/>
 <part name="GND49" library="supply1" deviceset="GND" device=""/>
@@
 <part name="GND47" library="supply1" deviceset="GND" device=""/>
 <part name="C43" library="rcl" deviceset="C-EU" device="C0805" value="100pF"/>
+<part name="JP10" library="pinhead" deviceset="PINHD-1X1" device=""/>
+<part name="JP11" library="pinhead" deviceset="PINHD-1X2" device=""/>
 </parts>
 <sheets>
@@
 <instance part="JP9" gate="A" x="215.9" y="-30.48"/>
 <instance part="C42" gate="G$1" x="165.1" y="5.08" rot="R90"/>
-<instance part="JP10" gate="G$1" x="-205.74" y="73.66" rot="R180"/>
 <instance part="GND53" gate="1" x="-195.58" y="63.5"/>
 <instance part="GND49" gate="1" x="35.56" y="38.1" rot="R90"/>
@@
 <instance part="GND47" gate="1" x="50.8" y="-33.02"/>
 <instance part="C43" gate="G$1" x="-5.08" y="38.1" rot="R90"/>
+<instance part="JP10" gate="G$1" x="-205.74" y="73.66" rot="R180"/>
+<instance part="JP11" gate="G$1" x="162.56" y="170.18"/>
 </instances>
 <busses>
@@
 </segment>
 <segment>
-<pinref part="JP10" gate="G$1" pin="2"/>
-<pinref part="GND53" gate="1" pin="GND"/>
-<wire x1="-203.2" y1="73.66" x2="-195.58" y2="73.66" width="0" layer="91"/>
-<wire x1="-195.58" y1="73.66" x2="-195.58" y2="71.12" width="0" layer="91"/>
-<pinref part="JP10" gate="G$1" pin="1"/>
-<wire x1="-195.58" y1="71.12" x2="-195.58" y2="66.04" width="0" layer="91"/>
-<wire x1="-203.2" y1="71.12" x2="-195.58" y2="71.12" width="0" layer="91"/>
-<junction x="-195.58" y="71.12"/>
-</segment>
-<segment>
 <pinref part="C27" gate="G$1" pin="2"/>
 <pinref part="GND49" gate="1" pin="GND"/>
@@
 <pinref part="GND47" gate="1" pin="GND"/>
 <wire x1="50.8" y1="-30.48" x2="50.8" y2="-25.4" width="0.1524" layer="91"/>
+</segment>
+<segment>
+<pinref part="JP10" gate="G$1" pin="1"/>
+<wire x1="-203.2" y1="73.66" x2="-195.58" y2="73.66" width="0.1524" layer="91"/>
+<pinref part="GND53" gate="1" pin="GND"/>
+<wire x1="-195.58" y1="73.66" x2="-195.58" y2="66.04" width="0.1524" layer="91"/>
 </segment>
 </net>
@@
 <net name="N$51" class="0">
 <segment>
-<wire x1="205.74" y1="-22.86" x2="205.74" y2="172.72" width="0.1524" layer="91"/>
 <pinref part="G1" gate="G$1" pin="+VIN"/>
-<wire x1="205.74" y1="172.72" x2="147.32" y2="172.72" width="0.1524" layer="91"/>
-<pinref part="JP9" gate="A" pin="2"/>
-<wire x1="205.74" y1="-22.86" x2="213.36" y2="-22.86" width="0.1524" layer="91"/>
+<pinref part="JP11" gate="G$1" pin="1"/>
+<wire x1="147.32" y1="172.72" x2="160.02" y2="172.72" width="0.1524" layer="91"/>
 </segment>
 </net>
 <net name="N$52" class="0">
 <segment>
-<wire x1="200.66" y1="-20.32" x2="200.66" y2="162.56" width="0.1524" layer="91"/>
+<pinref part="JP11" gate="G$1" pin="2"/>
+<wire x1="160.02" y1="170.18" x2="152.4" y2="170.18" width="0.1524" layer="91"/>
+<wire x1="152.4" y1="170.18" x2="152.4" y2="162.56" width="0.1524" layer="91"/>
 <pinref part="G1" gate="G$1" pin="-VIN"/>
-<wire x1="200.66" y1="162.56" x2="147.32" y2="162.56" width="0.1524" layer="91"/>
-<pinref part="JP9" gate="A" pin="1"/>
-<wire x1="200.66" y1="-20.32" x2="213.36" y2="-20.32" width="0.1524" layer="91"/>
-</segment>
-</net>
+<wire x1="152.4" y1="162.56" x2="147.32" y2="162.56" width="0.1524" layer="91"/>
+</segment>
+</net>

Commit message: Better comps
Parts:
- C1, C10, C11, C12, C13, C14, C15, C16, C17, C18, C19, C2, C20, C21, C22, C23, C24, C25, C26, C27, C3, C31, C32, C36, C37, C38, C4, C41, C42, C5, C6, C7, C8, C9: value 0.1uF -> 100nF; device rcl:C-EUC0805 -> SparkFun-Passives:CAP0805
- C29, C30, C43: device rcl:C-EUC0805 -> SparkFun-Passives:CAP0805
- R1, R10, R11, R12, R13, R14, R15, R16, R17, R18, R19, R2, R20, R21, R22, R23, R24, R25, R26, R27, R28, R3, R4, R5, R6, R7, R8, R9: device rcl:R-EU_R0805 -> SparkFun-Passives:RESISTOR0805-RES
