File: Adc.brd (EAGLE design)
At the start: 160 x 100 mm, 4 parts, among them IC1 ADS1256IDBT, IC2 ADUM1402ARWZ, IC3 AD8605ARTZ

Commit message: .
Parts:
- added C1, C10, C11, C12, C13, C14, C15, C16, C17, C18, C19, C2, C20, C21, C22, C23, C24, C25, C26, C27, C3, C31, C32, C36, C37, C38, C4, C41, C42, C5, C6, C7, C8, C9: 0.1uF, rcl:C0805
- added C28, C33, C34, C35, C39, C40: 47uF, rcl:E2-4
- added C29, C30: 18pF, rcl:C0805
- added IC10, IC4, IC5, IC6, IC7, IC8, IC9: AD8605ARTZ, nanoeeg:AD8605ARTZ
- added IC11: REF3125AIDBZT, nanoeeg:REF3125AIDBZT
- added IC12: MCP170333MB, linear:SOT89
- added JP1, JP2, JP3, JP4, JP5, JP6, JP7, JP8: (no value), pinhead:1X04
- added JP10: (no value), pinhead:1X02
- added JP9: (no value), pinhead:1X08
- added L1, L2, L3: (no value), rcl:L4532P
- added Q1: 8MHz, crystal:HC49U-V
- added R1, R10, R13, R16, R19, R22, R25, R26, R27, R28, R4, R7: 100, rcl:R0805
- added R11, R12, R14, R15, R17, R18, R2, R20, R21, R23, R24, R3, R5, R6, R8, R9: 1k, rcl:R0805
- moved G1 126.4 mm to (82.5, 91.4), turned to 270 degrees
- moved IC2 113.1 mm to (61.0, 71.1)
- moved IC1 54.7 mm to (29.2, 48.3)
- moved IC3 45.8 mm to (20.3, 21.6), turned to 180 degrees
Connections:
- removed net +VS: IC3.5
- removed net -VS: IC3.2
- new net +3.3V: C27.1, C35.+, C36.1, C41.2, IC1.14, IC1.15, IC1.16, IC12.3, IC2.1, IC2.7
- new net +5VA: C11.1, C14.1, C17.1, C2.1, C20.1, C23.1, C25.2, C37.1, C39.+, C5.1, C8.1, IC1.1, IC10.5, IC11.1, IC3.5, IC4.5, IC5.5, IC6.5, IC7.5, IC8.5, IC9.5, JP1.3, JP2.3, JP3.3, JP4.3, JP5.3, JP6.3, JP7.3, JP8.3, L1.1
- new net -5VA: C38.2, C40.-, JP1.4, JP2.4, JP3.4, JP4.4, JP5.4, JP6.4, JP7.4, JP8.4, L2.1
- new net GND: C1.1, C10.1, C11.2, C12.2, C13.1, C14.2, C15.2, C16.1, C17.2, C18.2, C19.1, C2.2, C20.2, C21.2, C22.1, C23.2, C24.2, C25.1, C26.2, C28.-, C3.2, C37.2, C38.1, C39.-, C4.1, C40.+, C5.2, C6.2, C7.1, C8.2, C9.2, IC1.2, IC1.3, IC10.2, IC11.3, IC3.2, IC4.2, IC5.2, IC6.2, IC7.2, IC8.2, IC9.2, JP1.2, JP10.1, JP10.2, JP2.2, JP3.2, JP4.2, JP5.2, JP6.2, JP7.2, JP8.2, L3.1
- new net GNDIO: C27.2, C29.2, C30.2, C31.2, C32.1, C33.-, C34.+, C35.-, C36.2, C41.1, G1.6, IC1.17, IC1.20, IC12.1, IC2.2, IC2.8, L3.2
- new net N$1: IC3.4, R2.2, R3.2
- new net N$10: IC5.1, R7.1, R9.1
- new net N$11: C9.1, IC1.8, R7.2
- new net N$12: JP3.1, R8.1
- new net N$13: IC6.4, R11.2, R12.2
- new net N$14: IC6.1, R10.1, R12.1
- new net N$15: C12.1, IC1.9, R10.2
- new net N$16: JP4.1, R11.1
- new net N$17: IC7.4, R14.2, R15.2
- new net N$18: IC7.1, R13.1, R15.1
- new net N$19: C15.1, IC1.10, R13.2
- new net N$2: IC3.1, R1.1, R3.1
- new net N$20: JP5.1, R14.1
- new net N$21: IC8.4, R17.2, R18.2
- new net N$22: IC8.1, R16.1, R18.1
- new net N$23: C18.1, IC1.11, R16.2
- new net N$24: JP6.1, R17.1
- new net N$25: IC9.4, R20.2, R21.2
- new net N$26: IC9.1, R19.1, R21.1
- new net N$27: C21.1, IC1.12, R19.2
- new net N$28: JP7.1, R20.1
- new net N$29: IC10.4, R23.2, R24.2
- new net N$3: JP1.1, R2.1
- new net N$30: IC10.1, R22.1, R24.1
- new net N$31: C24.1, IC1.13, R22.2
- new net N$32: JP8.1, R23.1
- new net N$33: C29.1, IC1.18, Q1.1
- new net N$34: C30.1, IC1.19, Q1.2
- new net N$35: IC2.11, JP9.7
- new net N$36: IC1.21, R25.1
- new net N$37: IC1.24, R26.1
- new net N$38: IC1.23, R27.1
- new net N$39: IC1.22, R28.1
- new net N$4: C3.1, IC1.6, R1.2
- new net N$40: C42.1, IC2.15, IC2.9, JP9.8
- new net N$41: C31.1, C33.+, G1.7, IC12.2@1, L1.2
- new net N$42: C32.2, C34.-, G1.5, L2.2
- new net N$43: C42.2, IC2.10, IC2.16, JP9.3
- new net N$44: IC2.3, R25.2
- new net N$45: IC2.4, R28.2
- new net N$46: IC2.5, R26.2
- new net N$47: IC2.6, R27.2
- new net N$48: IC2.12, JP9.6
- new net N$49: IC2.13, JP9.5
- new net N$5: IC4.4, R5.2, R6.2
- new net N$50: IC2.14, JP9.4
- new net N$51: G1.1, JP9.1
- new net N$52: G1.2, JP9.2
- new net N$6: IC4.1, R4.1, R6.1
- new net N$7: C6.1, IC1.7, R4.2
- new net N$8: JP2.1, R5.1
- new net N$9: IC5.4, R8.2, R9.2
- new net REF: C1.2, C10.2, C13.2, C16.2, C19.2, C22.2, C26.1, C28.+, C4.2, C7.2, IC1.4, IC1.5, IC10.3, IC11.2, IC3.3, IC4.3, IC5.3, IC6.3, IC7.3, IC8.3, IC9.3
Other:
- board size 160 x 100 mm -> 120.6 x 100 mm

Commit message: Rename lbr
Parts:
- G1: device nanoeeg:TMV0505D -> femtoexg:TMV0505D
- IC1: device nanoeeg:ADS1256IDBT -> femtoexg:ADS1256IDBT
- IC10, IC3, IC4, IC5, IC6, IC7, IC8, IC9: device nanoeeg:AD8605ARTZ -> femtoexg:AD8605ARTZ
- IC11: device nanoeeg:REF3125AIDBZT -> femtoexg:REF3125AIDBZT
- IC2: device nanoeeg:ADUM1402ARWZ -> femtoexg:ADUM1402ARWZ
Changed lines of the file:
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@@
 </autorouter>
 <elements>
-<element name="IC1" library="nanoeeg" package="ADS1256IDBT" value="ADS1256IDBT" x="29.21" y="48.26"/>
-<element name="IC2" library="nanoeeg" package="ADUM1402ARWZ" value="ADUM1402ARWZ" x="60.96" y="71.12"/>
-<element name="G1" library="nanoeeg" package="TMV0505D" value="TMV0505D" x="82.55" y="91.44" rot="R270"/>
-<element name="IC3" library="nanoeeg" package="AD8605ARTZ" value="AD8605ARTZ" x="20.32" y="21.59" rot="R180"/>
+<element name="IC1" library="femtoexg" package="ADS1256IDBT" value="ADS1256IDBT" x="29.21" y="48.26"/>
+<element name="IC2" library="femtoexg" package="ADUM1402ARWZ" value="ADUM1402ARWZ" x="60.96" y="71.12"/>
+<element name="G1" library="femtoexg" package="TMV0505D" value="TMV0505D" x="82.55" y="91.44" rot="R270"/>
+<element name="IC3" library="femtoexg" package="AD8605ARTZ" value="AD8605ARTZ" x="20.32" y="21.59" rot="R180"/>
 <element name="C1" library="rcl" package="C0805" value="0.1uF" x="19.05" y="26.67" rot="R270"/>
 <element name="C2" library="rcl" package="C0805" value="0.1uF" x="21.59" y="26.67" rot="R90"/>
@@
 <element name="C3" library="rcl" package="C0805" value="0.1uF" x="20.32" y="33.02" rot="R270"/>
 <element name="JP1" library="pinhead" package="1X04" value="" x="16.51" y="8.89" rot="R270"/>
-<element name="IC4" library="nanoeeg" package="AD8605ARTZ" value="AD8605ARTZ" x="30.48" y="21.59" rot="R180"/>
+<element name="IC4" library="femtoexg" package="AD8605ARTZ" value="AD8605ARTZ" x="30.48" y="21.59" rot="R180"/>
 <element name="C4" library="rcl" package="C0805" value="0.1uF" x="29.21" y="26.67" rot="R270"/>
 <element name="C5" library="rcl" package="C0805" value="0.1uF" x="31.75" y="26.67" rot="R90"/>
@@
 <element name="C6" library="rcl" package="C0805" value="0.1uF" x="30.48" y="33.02" rot="R270"/>
 <element name="JP2" library="pinhead" package="1X04" value="" x="26.67" y="8.89" rot="R270"/>
-<element name="IC5" library="nanoeeg" package="AD8605ARTZ" value="AD8605ARTZ" x="40.64" y="21.59" rot="R180"/>
+<element name="IC5" library="femtoexg" package="AD8605ARTZ" value="AD8605ARTZ" x="40.64" y="21.59" rot="R180"/>
 <element name="C7" library="rcl" package="C0805" value="0.1uF" x="39.37" y="26.67" rot="R270"/>
 <element name="C8" library="rcl" package="C0805" value="0.1uF" x="41.91" y="26.67" rot="R90"/>
@@
 <element name="C9" library="rcl" package="C0805" value="0.1uF" x="40.64" y="33.02" rot="R270"/>
 <element name="JP3" library="pinhead" package="1X04" value="" x="36.83" y="8.89" rot="R270"/>
-<element name="IC6" library="nanoeeg" package="AD8605ARTZ" value="AD8605ARTZ" x="50.8" y="21.59" rot="R180"/>
+<element name="IC6" library="femtoexg" package="AD8605ARTZ" value="AD8605ARTZ" x="50.8" y="21.59" rot="R180"/>
 <element name="C10" library="rcl" package="C0805" value="0.1uF" x="49.53" y="26.67" rot="R270"/>
 <element name="C11" library="rcl" package="C0805" value="0.1uF" x="52.07" y="26.67" rot="R90"/>
@@
 <element name="C12" library="rcl" package="C0805" value="0.1uF" x="50.8" y="33.02" rot="R270"/>
 <element name="JP4" library="pinhead" package="1X04" value="" x="46.99" y="8.89" rot="R270"/>
-<element name="IC7" library="nanoeeg" package="AD8605ARTZ" value="AD8605ARTZ" x="60.96" y="21.59" rot="R180"/>
+<element name="IC7" library="femtoexg" package="AD8605ARTZ" value="AD8605ARTZ" x="60.96" y="21.59" rot="R180"/>
 <element name="C13" library="rcl" package="C0805" value="0.1uF" x="59.69" y="26.67" rot="R270"/>
 <element name="C14" library="rcl" package="C0805" value="0.1uF" x="62.23" y="26.67" rot="R90"/>
@@
 <element name="C15" library="rcl" package="C0805" value="0.1uF" x="60.96" y="33.02" rot="R270"/>
 <element name="JP5" library="pinhead" package="1X04" value="" x="57.15" y="8.89" rot="R270"/>
-<element name="IC8" library="nanoeeg" package="AD8605ARTZ" value="AD8605ARTZ" x="71.12" y="21.59" rot="R180"/>
+<element name="IC8" library="femtoexg" package="AD8605ARTZ" value="AD8605ARTZ" x="71.12" y="21.59" rot="R180"/>
 <element name="C16" library="rcl" package="C0805" value="0.1uF" x="69.85" y="26.67" rot="R270"/>
 <element name="C17" library="rcl" package="C0805" value="0.1uF" x="72.39" y="26.67" rot="R90"/>
@@
 <element name="C18" library="rcl" package="C0805" value="0.1uF" x="71.12" y="33.02" rot="R270"/>
 <element name="JP6" library="pinhead" package="1X04" value="" x="67.31" y="8.89" rot="R270"/>
-<element name="IC9" library="nanoeeg" package="AD8605ARTZ" value="AD8605ARTZ" x="81.28" y="21.59" rot="R180"/>
+<element name="IC9" library="femtoexg" package="AD8605ARTZ" value="AD8605ARTZ" x="81.28" y="21.59" rot="R180"/>
 <element name="C19" library="rcl" package="C0805" value="0.1uF" x="80.01" y="26.67" rot="R270"/>
 <element name="C20" library="rcl" package="C0805" value="0.1uF" x="82.55" y="26.67" rot="R90"/>
@@
 <element name="C21" library="rcl" package="C0805" value="0.1uF" x="81.28" y="33.02" rot="R270"/>
 <element name="JP7" library="pinhead" package="1X04" value="" x="77.47" y="8.89" rot="R270"/>
-<element name="IC10" library="nanoeeg" package="AD8605ARTZ" value="AD8605ARTZ" x="91.44" y="21.59" rot="R180"/>
+<element name="IC10" library="femtoexg" package="AD8605ARTZ" value="AD8605ARTZ" x="91.44" y="21.59" rot="R180"/>
 <element name="C22" library="rcl" package="C0805" value="0.1uF" x="90.17" y="26.67" rot="R270"/>
 <element name="C23" library="rcl" package="C0805" value="0.1uF" x="92.71" y="26.67" rot="R90"/>
@@
 <element name="C27" library="rcl" package="C0805" value="0.1uF" x="33.02" y="54.61" rot="R180"/>
 <element name="C28" library="rcl" package="E2-4" value="47uF" x="33.02" y="62.23"/>
-<element name="IC11" library="nanoeeg" package="REF3125AIDBZT" value="REF3125AIDBZT" x="34.29" y="71.12"/>
+<element name="IC11" library="femtoexg" package="REF3125AIDBZT" value="REF3125AIDBZT" x="34.29" y="71.12"/>
 <element name="Q1" library="crystal" package="HC49U-V" value="8MHz" x="21.59" y="57.15" rot="R180">
 <attribute name="OC_NEWARK" value="unknown" x="21.59" y="57.15" size="1.778" layer="27" rot="R180" display="off"/>

Commit message: Dimensions
Parts:
- removed L3: (no value), rcl:L4532P
- added C43: 100pF, rcl:C0805
- moved JP9 109.7 mm to (16.5, 27.9), turned to 180 degrees
- moved G1 85.1 mm to (30.5, 24.1), turned to 90 degrees
- moved C33 78.1 mm to (43.2, 23.5), turned to 90 degrees
- moved C31 73.9 mm to (45.1, 23.5), flipped to the bottom, turned to 90 degrees
- moved C35 73.4 mm to (48.3, 15.2)
- moved L1 72.5 mm to (50.8, 23.5), turned to 180 degrees
- moved C3 71.8 mm to (90.2, 16.5), flipped to the bottom
- moved C30 70.3 mm to (84.5, 38.7), flipped to the bottom, turned to 0 degrees
- moved IC2 70.1 mm to (13.3, 19.7), flipped to the bottom
- moved C41 70.1 mm to (6.35, 15.2), turned to 270 degrees
- moved C39 69.6 mm to (58.4, 23.5), turned to 90 degrees
- moved C37 69.2 mm to (56.5, 23.5), flipped to the bottom, turned to 90 degrees
- moved C42 68.1 mm to (16.5, 24.1), turned to 90 degrees
- moved C36 67.7 mm to (53.3, 20.3), flipped to the bottom, turned to 180 degrees
- moved C32 64.9 mm to (45.1, 27.9), flipped to the bottom, turned to 90 degrees
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Connections:
- removed net GNDIO: C27.2, C29.2, C30.2, C31.2, C32.1, C33.-, C34.+, C35.-, C36.2, C41.1, G1.6, IC1.17, IC1.20, IC12.1, IC2.2, IC2.8, L3.2
- net GND: now also C27.2, C29.2, C30.2, C31.2, C32.1, C33.-, C34.+, C35.-, C36.2, C41.1, C43.2, G1.6, IC1.17, IC1.20, IC12.1, IC2.2, IC2.8; no longer L3.1
- net N$51: now also JP9.2; no longer JP9.1
- net N$52: now also JP9.1; no longer JP9.2
- net REF: now also C43.1
Routing:
- net GND: track 0.00 -> 201.2 mm, vias 0 -> 1
- net REF: track 0.00 -> 134.7 mm, vias 0 -> 8
- net +5VA: track 0.00 -> 131.0 mm, vias 0 -> 2
- net -5VA: track 0.00 -> 77.4 mm, vias 0 -> 1
- net N$43: track 0.00 -> 28.3 mm, vias 0 -> 2
- net N$40: track 0.00 -> 25.3 mm, vias 0 -> 2
- net N$29: track 0.00 -> 12.7 mm
- net N$9: track 0.00 -> 12.7 mm
- net N$5: track 0.00 -> 12.7 mm
- net N$17: track 0.00 -> 12.7 mm
- net N$1: track 0.00 -> 12.7 mm
- net N$21: track 0.00 -> 12.7 mm
- net N$13: track 0.00 -> 12.7 mm
- net N$25: track 0.00 -> 12.7 mm
- net N$41: track 0.00 -> 9.78 mm, vias 0 -> 1
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Other:
- board size 120.6 x 100 mm -> 96.8 x 31.3 mm

Commit message: Routing
Parts:
- added JP11: (no value), pinhead:1X02
- JP10: device pinhead:1X02 -> pinhead:1X01
- Q1: value 8MHz -> 7.68MHz
- moved C6 94.0 mm to (-6.35, 16.5), turned to 0 degrees
- moved C9 91.4 mm to (-6.35, 17.8), flipped to the top, turned to 180 degrees
- moved C12 88.9 mm to (-6.35, 19.1), turned to 0 degrees
- moved C15 86.4 mm to (-6.35, 20.3), flipped to the top, turned to 180 degrees
- moved C3 86.4 mm to (3.81, 20.3), turned to 0 degrees
- moved C18 84.0 mm to (-6.35, 21.6), turned to 0 degrees
- moved C21 81.5 mm to (-6.35, 22.9), flipped to the top, turned to 180 degrees
- moved C24 79.1 mm to (-6.35, 24.1), turned to 0 degrees
- moved IC11 76.2 mm to (3.81, 10.2), turned to 90 degrees
- moved IC1 71.5 mm to (12.7, 17.1), turned to 90 degrees
- moved C26 68.6 mm to (3.81, 14.6), turned to 180 degrees
- moved C43 68.3 mm to (6.99, 14.0), turned to 270 degrees
- moved C25 67.6 mm to (6.99, 10.2), flipped to the bottom, turned to 270 degrees
- moved C28 67.6 mm to (3.81, 12.7), turned to 0 degrees
- moved Q1 65.1 mm to (21.0, 19.7)
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Connections:
- net GND: no longer JP10.2
- net N$51: now also JP11.1; no longer JP9.2
- net N$52: now also JP11.2; no longer JP9.1
Routing:
- net N$31: track 0.00 -> 70.4 mm
- net N$27: track 0.00 -> 68.2 mm
- net N$23: track 0.00 -> 58.4 mm
- net N$19: track 0.00 -> 48.6 mm
- net N$15: track 0.00 -> 38.8 mm
- net N$11: track 0.00 -> 29.0 mm
- net N$43: track 28.3 -> 0.00 mm, vias 2 -> 0
- net N$40: track 25.3 -> 0.00 mm, vias 2 -> 0
- net N$4: track 0.00 -> 23.7 mm, vias 0 -> 1
- net REF: track 134.7 -> 156.3 mm
- net N$7: track 0.00 -> 21.5 mm
- net +5VA: track 131.0 -> 152.2 mm
- net GND: track 201.2 -> 221.5 mm
- net +3.3V: track 0.00 -> 7.90 mm
- net N$50: track 5.08 -> 0.00 mm
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Other:
- board size 96.8 x 31.3 mm -> 96.8 x 28.7 mm

Commit message: Better comps
Parts:
- C1, C10, C11, C12, C13, C14, C15, C16, C17, C18, C19, C2, C20, C21, C22, C23, C24, C25, C26, C27, C3, C31, C32, C36, C37, C38, C4, C41, C42, C5, C6, C7, C8, C9: value 0.1uF -> 100nF; device rcl:C0805 -> SparkFun-Passives:0805
- C29, C30, C43: device rcl:C0805 -> SparkFun-Passives:0805
- R1, R10, R11, R12, R13, R14, R15, R16, R17, R18, R19, R2, R20, R21, R22, R23, R24, R25, R26, R27, R28, R3, R4, R5, R6, R7, R8, R9: device rcl:R0805 -> SparkFun-Passives:0805
- moved R25 23.4 mm to (38.1, 19.1)
- moved C24 22.2 mm to (-6.35, 1.91), flipped to the top, turned to 180 degrees
- moved C41 19.7 mm to (53.3, 30.5), turned to 0 degrees
- moved C21 19.1 mm to (-6.35, 3.81)
- moved R28 19.1 mm to (41.9, 22.9)
- moved R27 18.8 mm to (41.9, 20.3)
- moved C18 15.9 mm to (-6.35, 5.71), flipped to the top, turned to 180 degrees
- moved C29 14.7 mm to (19.1, 22.9)
- moved C30 14.7 mm to (22.9, 22.9)
- moved R26 13.5 mm to (38.1, 21.6)
- moved C15 12.7 mm to (-6.35, 7.62)
- moved C3 11.4 mm to (-6.35, 15.2), flipped to the top, turned to 180 degrees
- moved C27 11.0 mm to (14.0, 24.1), turned to 0 degrees
- moved C12 9.53 mm to (-6.35, 9.53), flipped to the top, turned to 180 degrees
- moved C36 9.25 mm to (36.8, 24.1), flipped to the top, turned to 0 degrees
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Routing:
- net N$31: track 70.4 -> 0.00 mm
- net N$27: track 68.2 -> 0.00 mm
- net N$23: track 58.4 -> 0.00 mm
- net N$19: track 48.6 -> 0.00 mm
- net N$15: track 38.8 -> 0.00 mm
- net GND: track 221.5 -> 186.3 mm
- net N$11: track 29.0 -> 0.00 mm
- net N$7: track 21.5 -> 2.22 mm
- net REF: track 156.3 -> 137.8 mm
- net +5VA: track 152.2 -> 139.3 mm
- net N$30: track 5.58 -> 1.88 mm
- net N$26: track 5.58 -> 1.88 mm
- net N$6: track 5.58 -> 1.88 mm
- net N$2: track 5.58 -> 1.88 mm
- net N$14: track 5.58 -> 1.88 mm
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
Commit message: .
Routing:
- net +5VA: track 139.3 -> 150.0 mm
