File: InstAmp.brd (EAGLE design)
At the start: 77.5 x 54.3 mm, 37 parts, among them IC1 AD8221ARZ, IC2 TLC2254ID

Commit message: Rename lbr
Parts:
- IC1: device nanoeeg:AD8221ARZ -> femtoexg:AD8221ARZ
- IC2: device nanoeeg:TLC2254ID -> femtoexg:TLC2254ID
Changed lines of the file:
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@@
 <element name="R5" library="rcl" package="R0805" value="2k2" x="17.78" y="17.78" rot="MR180"/>
 <element name="R6" library="rcl" package="R0805" value="2k2" x="17.78" y="5.08" rot="MR180"/>
-<element name="IC1" library="nanoeeg" package="AD8221ARZ" value="AD8221ARZ" x="22.86" y="11.43" rot="MR90"/>
+<element name="IC1" library="femtoexg" package="AD8221ARZ" value="AD8221ARZ" x="22.86" y="11.43" rot="MR90"/>
 <element name="R7" library="rcl" package="R0805" value="2k" x="17.78" y="11.43" rot="MR270"/>
 <element name="C4" library="rcl" package="C0805" value="0.1" x="73.66" y="24.13"/>
 <element name="C5" library="rcl" package="C0805" value="0.1" x="60.96" y="44.45"/>
-<element name="IC2" library="nanoeeg" package="TLC2254ID" value="TLC2254ID" x="33.02" y="25.4" rot="R90"/>
+<element name="IC2" library="femtoexg" package="TLC2254ID" value="TLC2254ID" x="33.02" y="25.4" rot="R90"/>
 <element name="R8" library="rcl" package="R0805" value="100k" x="24.13" y="33.02"/>
 <element name="R9" library="rcl" package="R0805" value="100k" x="30.48" y="39.37"/>

Commit message: Dimensions
Parts:
- JP1: value (none) -> OUT
- moved R16 45.8 mm to (69.8, 2.54)
- moved C11 43.2 mm to (61.0, 10.2)
- moved IC2 39.9 mm to (69.8, 10.2)
- moved C6 36.2 mm to (61.6, 3.17)
- moved C4 28.7 mm to (53.3, 3.81)
- moved R17 28.1 mm to (61.6, 21.6)
- moved R9 27.0 mm to (48.3, 19.1)
- moved C5 25.3 mm to (68.6, 20.3)
- moved R14 24.2 mm to (54.0, 19.1)
- moved JP1 24.1 mm to (20.3, 7.62)
- moved R8 23.8 mm to (41.9, 17.1)
- moved D2 23.6 mm to (12.1, 6.35)
- moved R15 21.3 mm to (36.2, 20.3)
- moved R13 21.0 mm to (54.0, 8.26)
- moved C10 17.3 mm to (59.1, 17.1)
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Other:
- board size 77.5 x 54.3 mm -> 77.5 x 18 mm

Commit message: Routing
Parts:
- C4, C5, C6, C7: value 0.1 -> 0.1uF
- moved C5 58.5 mm to (19.1, -10.8), flipped to the bottom, turned to 270 degrees
- moved C11 41.8 mm to (24.1, -9.53), flipped to the bottom
- moved IC2 36.9 mm to (33.0, 8.89), flipped to the bottom, turned to 180 degrees
- moved C4 35.9 mm to (19.1, -6.67), flipped to the bottom, turned to 270 degrees
- moved R16 31.5 mm to (40.0, 12.7), turned to 90 degrees
- moved C6 31.0 mm to (33.0, 15.2), flipped to the bottom, turned to 90 degrees
- moved C1 29.7 mm to (5.71, -8.89)
- moved IC1 29.7 mm to (14.0, -8.89)
- moved R6 29.7 mm to (7.62, -5.71)
- moved R7 29.7 mm to (8.26, -8.89)
- moved R5 29.7 mm to (7.62, -12.1)
- moved R17 25.0 mm to (37.5, 15.2), flipped to the bottom, turned to 270 degrees
- moved R9 24.3 mm to (30.5, 2.54), flipped to the bottom, turned to 270 degrees
- moved C10 22.4 mm to (40.6, 4.45), flipped to the bottom, turned to 270 degrees
- moved R11 21.6 mm to (26.7, 15.2), flipped to the bottom, turned to 270 degrees
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Routing:
- net N$10: track 0.00 -> 1.27 mm
- net N$9: track 0.00 -> 1.27 mm

Commit message: Simplification of circuit
Parts:
- IC2: device femtoexg:TLC2254ID -> linear:SO14
- moved C9 12.7 mm to (24.1, 15.2), turned to 270 degrees
- moved C1 11.4 mm to (17.1, -9.53)
- moved R7 11.1 mm to (19.4, -9.53)
- moved IC1 10.8 mm to (24.8, -9.53)
- moved C11 10.8 mm to (34.9, -10.2)
- moved C4 10.8 mm to (29.8, -7.30)
- moved C5 10.8 mm to (29.8, -11.4)
- moved R5 10.8 mm to (18.4, -12.7)
- moved R6 10.8 mm to (18.4, -6.35)
- moved R10 3.42 mm to (46.4, 7.62)
- moved R13 1.80 mm to (41.3, 11.4)
- moved R16 1.80 mm to (38.7, 11.4), turned to 270 degrees
- moved R15 0.32 mm to (42.9, 4.45)
Connections:
- removed net N$14 (its old number): IC2.2, R11.2, R12.2
- removed net N$18: IC2.7, R13.1, R15.2, R16.1
- removed net N$22 (its old number): IC2.6, R16.2, R17.2
- new net N$10: IC2.6, R16.1, R17.2
- new net N$23: IC2.2, R11.1, R12.2
- new net N$9: IC2.7, R13.1, R15.2, R16.2
- net OUT: now also R11.2; no longer R11.1
Routing:
- net N$7: track 1.27 -> 0.00 mm
- net N$17: track 1.27 -> 0.00 mm

Commit message: Amp routing
Parts:
- moved JP1 0.63 mm to (22.9, 6.99)
Changed lines of the file:
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@@
 <element name="R16" library="rcl" package="R0805" value="910k" x="38.735" y="11.43" rot="R270"/>
 <element name="R17" library="rcl" package="R0805" value="100k" x="37.465" y="15.24" rot="MR270"/>
-<element name="JP1" library="pinhead" package="1X04/90" value="OUT" x="22.86" y="7.62" rot="R180"/>
+<element name="JP1" library="pinhead" package="1X04/90" value="OUT" x="22.86" y="6.985" rot="R180"/>
 <element name="IC2" library="linear" package="SO14" value="TLC2254ID" x="33.02" y="8.89" rot="MR180"/>
 </elements>
@@
 <wire x1="31.115" y1="16.19" x2="33.02" y2="16.19" width="0" layer="19" extent="16-16"/>
 <wire x1="28.8925" y1="16.19" x2="31.115" y2="16.19" width="0" layer="19" extent="16-16"/>
-<wire x1="24.13" y1="11.43" x2="28.8925" y2="16.19" width="0" layer="19" extent="16-16"/>
-<wire x1="30.48" y1="1.59" x2="24.13" y2="11.43" width="0" layer="19" extent="16-16"/>
+<wire x1="24.13" y1="10.795" x2="28.8925" y2="16.19" width="0" layer="19" extent="16-16"/>
+<wire x1="30.48" y1="1.59" x2="24.13" y2="10.795" width="0" layer="19" extent="16-16"/>
 <wire x1="33.02" y1="1.59" x2="30.48" y2="1.59" width="0" layer="19" extent="16-16"/>
 <wire x1="36.83" y1="1.59" x2="33.02" y2="1.59" width="0" layer="19" extent="16-16"/>
@@
 <wire x1="29.845" y1="-10.48" x2="29.845" y2="-8.2525" width="0" layer="19" extent="16-16"/>
 <wire x1="27.365" y1="-8.89" x2="29.845" y2="-8.2525" width="0" layer="19" extent="16-16"/>
-<wire x1="4.13" y1="5.715" x2="24.13" y2="11.43" width="0" layer="19" extent="16-16"/>
+<wire x1="4.13" y1="5.715" x2="24.13" y2="10.795" width="0" layer="19" extent="16-16"/>
 <wire x1="2.1" y1="5.715" x2="4.13" y2="5.715" width="0" layer="19" extent="16-16"/>
 <wire x1="4.13" y1="17.78" x2="4.13" y2="5.715" width="0" layer="19" extent="16-16"/>
@@
 <wire x1="29.845" y1="-6.3525" x2="33.02" y2="3.49" width="0" layer="19" extent="16-16"/>
 <wire x1="27.365" y1="-7.62" x2="29.845" y2="-6.3525" width="0" layer="19" extent="16-16"/>
-<wire x1="19.05" y1="11.43" x2="33.02" y2="6.29" width="0" layer="19" extent="16-16"/>
-<wire x1="13.015" y1="17.315" x2="19.05" y2="11.43" width="0" layer="19" extent="16-16"/>
+<wire x1="19.05" y1="10.795" x2="33.02" y2="6.29" width="0" layer="19" extent="16-16"/>
+<wire x1="13.015" y1="17.315" x2="19.05" y2="10.795" width="0" layer="19" extent="16-16"/>
 <wire x1="9.84" y1="15.41" x2="13.015" y2="17.315" width="0" layer="19" extent="16-16"/>
-<wire x1="13.015" y1="5.25" x2="19.05" y2="11.43" width="0" layer="19" extent="16-16"/>
+<wire x1="13.015" y1="5.25" x2="19.05" y2="10.795" width="0" layer="19" extent="16-16"/>
 <wire x1="9.84" y1="3.345" x2="13.015" y2="5.25" width="0" layer="19" extent="16-16"/>
 </signal>
@@
 <contactref element="IC2" pad="4"/>
 <wire x1="33.02" y1="11.49" x2="33.02" y2="14.29" width="0" layer="19" extent="16-16"/>
-<wire x1="21.59" y1="11.43" x2="33.02" y2="11.49" width="0" layer="19" extent="16-16"/>
-<wire x1="11.115" y1="17.315" x2="21.59" y2="11.43" width="0" layer="19" extent="16-16"/>
+<wire x1="21.59" y1="10.795" x2="33.02" y2="11.49" width="0" layer="19" extent="16-16"/>
+<wire x1="11.115" y1="17.315" x2="21.59" y2="10.795" width="0" layer="19" extent="16-16"/>
 <wire x1="7.94" y1="15.41" x2="11.115" y2="17.315" width="0" layer="19" extent="16-16"/>
 <wire x1="11.115" y1="5.25" x2="7.94" y2="15.41" width="0" layer="19" extent="16-16"/>
@@
 <contactref element="C9" pad="2"/>
 <wire x1="24.13" y1="14.29" x2="26.67" y2="14.29" width="0" layer="19" extent="1-16"/>
-<wire x1="26.67" y1="11.43" x2="26.67" y2="14.29" width="0" layer="19" extent="16-16"/>
-<wire x1="29.21" y1="11.49" x2="26.67" y2="11.43" width="0" layer="19" extent="16-16"/>
+<wire x1="26.67" y1="10.795" x2="26.67" y2="14.29" width="0" layer="19" extent="16-16"/>
+<wire x1="29.21" y1="11.49" x2="26.67" y2="10.795" width="0" layer="19" extent="16-16"/>
 </signal>
 <signal name="N$20">

Commit message: Better comps
Parts:
- removed IN+, IN-: 1503_09, con-lumberg:1503_09
- added +IN, -IN: (no value), SparkFun-Connectors:STEREOJACK2.5MM_SMD
- C1, C10, C11, C2, C3, C8, C9: device rcl:C0805 -> SparkFun-Passives:0805
- C4, C5, C6, C7: value 0.1uF -> 100nF; device rcl:C0805 -> SparkFun-Passives:0805
- R1, R10, R11, R12, R13, R14, R15, R16, R17, R2, R3, R4, R5, R6, R7, R8, R9: device rcl:R0805 -> SparkFun-Passives:0805
- moved C5 40.3 mm to (12.1, 24.8), flipped to the top, turned to 0 degrees
- moved C4 35.2 mm to (15.2, 24.8), flipped to the top, turned to 0 degrees
- moved C7 35.2 mm to (5.71, 24.8), flipped to the top, turned to 0 degrees
- moved R8 32.4 mm to (5.08, 8.89), flipped to the top, turned to 180 degrees
- moved R5 29.5 mm to (14.6, 16.5), flipped to the top, turned to 0 degrees
- moved C6 25.9 mm to (8.89, 24.8), flipped to the top, turned to 0 degrees
- moved R9 25.5 mm to (5.08, 0.64), flipped to the top, turned to 180 degrees
- moved C11 24.8 mm to (34.3, 14.6), turned to 270 degrees
- moved R10 22.4 mm to (27.9, 20.3), turned to 0 degrees
- moved R4 20.9 mm to (10.8, 1.27), flipped to the top, turned to 0 degrees
- moved C3 20.4 mm to (3.81, -2.54), flipped to the top, turned to 0 degrees
- moved D4 16.7 mm to (-3.81, 13.3)
- moved D2 16.3 mm to (-3.81, 2.54)
- moved R6 15.3 mm to (14.0, 8.26), flipped to the top, turned to 0 degrees
- moved C10 14.9 mm to (32.4, 16.8), turned to 180 degrees
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Connections:
- net GND: now also +IN.5, -IN.5; no longer IN+.1, IN-.1
- net N$1: now also -IN.1; no longer IN-.2
- net N$11: now also C10.1; no longer C11.2
- net N$2: now also -IN.4; no longer IN-.3
- net N$22: now also C11.2; no longer C10.1
- net N$3: now also +IN.1, R1.1; no longer IN+.3, R3.1
- net N$4: now also +IN.4, R3.1; no longer IN+.2, R1.1

Commit message: .
Parts:
- removed D3, D4: BAV199, diode:SOT23
- +IN, -IN: value (none) -> AUDIOJACK2.5-SMD; device SparkFun-Connectors:STEREOJACK2.5MM_SMD -> femtoexg:AUDIOJACK2.5-SMD
- D1, D2: device diode:SOT23 -> SparkFun-DiscreteSemi:SOT23
- moved D1 20.5 mm to (14.0, -3.17), turned to 180 degrees
- moved D2 15.7 mm to (10.8, -3.17)
- moved C1 15.4 mm to (15.2, 7.62), turned to 270 degrees
- moved C2 13.6 mm to (13.3, 9.53), turned to 270 degrees
- moved C3 12.6 mm to (13.3, 5.71), turned to 270 degrees
- moved R17 9.09 mm to (36.2, 14.6), flipped to the bottom, turned to 270 degrees
- moved C5 8.64 mm to (19.1, 19.7), turned to 180 degrees
- moved R8 8.54 mm to (10.8, 15.2), turned to 0 degrees
- moved R9 8.08 mm to (10.8, 6.35), turned to 0 degrees
- moved C10 7.96 mm to (39.7, 13.7), turned to 90 degrees
- moved R13 6.98 mm to (36.2, 17.1)
- moved R1 6.79 mm to (9.53, 9.84)
- moved R2 6.79 mm to (9.53, 0.95)
- moved R3 6.79 mm to (9.53, 16.8)
- moved R4 6.79 mm to (9.53, 7.94)
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Connections:
- net +5V: no longer D3.2, D4.2
- net -5V: no longer D3.1, D4.1
- net GND: now also +IN.GND1, +IN.GND2, +IN.SW, -IN.GND1, -IN.GND2, -IN.SW; no longer +IN.5, -IN.5
- net N$1: now also +IN.L, R1.1; no longer -IN.1, R2.1
- net N$17: no longer D2.3
- net N$2: now also -IN.R; no longer -IN.4
- net N$3: now also +IN.R, R3.1; no longer +IN.1, R1.1
- net N$4: now also -IN.L, R2.1; no longer +IN.4, R3.1
- net N$5: now also D2.3; no longer D3.3
- net N$7: no longer D4.3
Routing:
- net GND: track 0.00 -> 31.5 mm

Commit message: .
Parts:
- moved C7 32.4 mm to (36.2, 1.27), turned to 180 degrees
- moved C6 32.4 mm to (39.4, 1.27), turned to 180 degrees
- moved C10 19.0 mm to (23.8, 3.17), turned to 180 degrees
- moved C5 17.9 mm to (24.1, 2.54), turned to 270 degrees
- moved C4 16.2 mm to (24.1, 5.71), turned to 270 degrees
- moved D2 14.5 mm to (6.99, 10.8), turned to 90 degrees
- moved D1 12.3 mm to (6.99, 6.99), turned to 90 degrees
- moved R5 10.3 mm to (12.7, 1.27), flipped to the bottom, turned to 180 degrees
- moved +IN 8.89 mm to (1.27, 4.45)
- moved -IN 8.89 mm to (1.27, 13.3)
- moved R3 8.89 mm to (9.53, 7.94)
- moved R4 8.89 mm to (9.53, 16.8)
- moved R8 8.89 mm to (10.8, 6.35)
- moved R9 8.89 mm to (10.8, 15.2)
- moved R1 8.89 mm to (9.53, 0.95)
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Routing:
- net GND: track 31.5 -> 55.3 mm, vias 0 -> 1
- net +5V: track 0.00 -> 19.1 mm
- net -5V: track 0.00 -> 16.2 mm
- net N$6: track 0.00 -> 11.5 mm, vias 0 -> 1
- net N$5: track 0.00 -> 9.14 mm, vias 0 -> 1
- net N$8: track 0.00 -> 2.63 mm
- net N$16: track 0.00 -> 2.63 mm
- net N$12: track 0.00 -> 2.48 mm
- net N$7: track 0.00 -> 1.81 mm
- net N$17: track 0.00 -> 1.81 mm
- net N$2: track 0.00 -> 1.61 mm
- net N$4: track 0.00 -> 1.61 mm
- net N$3: track 0.00 -> 1.61 mm
- net N$1: track 0.00 -> 1.61 mm
Other:
- board size 77.5 x 18 mm -> 41.3 x 18 mm
