File: InstAmp.sch (EAGLE design)
At the start: 37 parts, among them IC1 AD8221ARZ, IC2 TLC2254ID

Commit message: Rename lbr
Parts:
- IC1: device nanoeeg:AD8221ARZ -> femtoexg:AD8221ARZ
- IC2: device nanoeeg:TLC2254ID -> femtoexg:TLC2254ID
Changed lines of the file:
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@@
 <part name="R5" library="rcl" deviceset="R-EU_" device="R0805" value="2k2"/>
 <part name="R6" library="rcl" deviceset="R-EU_" device="R0805" value="2k2"/>
-<part name="IC1" library="nanoeeg" deviceset="AD8221ARZ" device=""/>
+<part name="IC1" library="femtoexg" deviceset="AD8221ARZ" device=""/>
 <part name="R7" library="rcl" deviceset="R-EU_" device="R0805" value="2k"/>
 <part name="GND4" library="supply1" deviceset="GND" device=""/>
@@
 <part name="GND5" library="supply1" deviceset="GND" device=""/>
 <part name="GND6" library="supply1" deviceset="GND" device=""/>
-<part name="IC2" library="nanoeeg" deviceset="TLC2254ID" device=""/>
+<part name="IC2" library="femtoexg" deviceset="TLC2254ID" device=""/>
 <part name="R8" library="rcl" deviceset="R-EU_" device="R0805" value="100k"/>
 <part name="R9" library="rcl" deviceset="R-EU_" device="R0805" value="100k"/>

Commit message: Dimensions
Parts:
- JP1: value (none) -> OUT
Changed lines of the file:
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@@
 <setting verticaltext="up"/>
 </settings>
-<grid distance="0.1" unitdist="inch" unit="inch" style="dots" multiple="1" display="yes" altdistance="0.01" altunitdist="inch" altunit="inch"/>
+<grid distance="0.1" unitdist="inch" unit="inch" style="lines" multiple="1" display="no" altdistance="0.01" altunitdist="inch" altunit="inch"/>
 <layers>
 <layer number="1" name="Top" color="4" fill="9" visible="no" active="no"/>
@@
 <part name="R17" library="rcl" deviceset="R-EU_" device="R0805" value="100k"/>
 <part name="GND14" library="supply1" deviceset="GND" device=""/>
-<part name="JP1" library="pinhead" deviceset="PINHD-1X4" device="/90"/>
+<part name="JP1" library="pinhead" deviceset="PINHD-1X4" device="/90" value="OUT"/>
 <part name="GND15" library="supply1" deviceset="GND" device=""/>
 </parts>
@@
 <wire x1="284.48" y1="-119.38" x2="284.48" y2="-121.92" width="0.1524" layer="91"/>
 <label x="284.48" y="-121.92" size="1.778" layer="95" rot="R270" xref="yes"/>
+<junction x="284.48" y="-119.38"/>
 </segment>
 <segment>
@@
 <wire x1="284.48" y1="17.78" x2="284.48" y2="20.32" width="0.1524" layer="91"/>
 <label x="284.48" y="20.32" size="1.778" layer="95" rot="R90" xref="yes"/>
+<junction x="284.48" y="17.78"/>
 </segment>
 <segment>
@@
 </sheet>
 </sheets>
+<errors>
+</errors>
 </schematic>
 </drawing>

Commit message: Routing
Parts:
- C4, C5, C6, C7: value 0.1 -> 0.1uF
Changed lines of the file:
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@@
 <part name="R7" library="rcl" deviceset="R-EU_" device="R0805" value="2k"/>
 <part name="GND4" library="supply1" deviceset="GND" device=""/>
-<part name="C4" library="rcl" deviceset="C-EU" device="C0805" value="0.1"/>
-<part name="C5" library="rcl" deviceset="C-EU" device="C0805" value="0.1"/>
+<part name="C4" library="rcl" deviceset="C-EU" device="C0805" value="0.1uF"/>
+<part name="C5" library="rcl" deviceset="C-EU" device="C0805" value="0.1uF"/>
 <part name="GND5" library="supply1" deviceset="GND" device=""/>
 <part name="GND6" library="supply1" deviceset="GND" device=""/>
@@
 <part name="GND7" library="supply1" deviceset="GND" device=""/>
 <part name="GND8" library="supply1" deviceset="GND" device=""/>
-<part name="C6" library="rcl" deviceset="C-EU" device="C0805" value="0.1"/>
-<part name="C7" library="rcl" deviceset="C-EU" device="C0805" value="0.1"/>
+<part name="C6" library="rcl" deviceset="C-EU" device="C0805" value="0.1uF"/>
+<part name="C7" library="rcl" deviceset="C-EU" device="C0805" value="0.1uF"/>
 <part name="GND9" library="supply1" deviceset="GND" device=""/>
 <part name="GND10" library="supply1" deviceset="GND" device=""/>

Commit message: Simplification of circuit
Parts:
- IC2: device femtoexg:TLC2254ID -> linear:4AMP_P4+11D
Connections:
- removed net N$11 (its old number): C8.1, IC2.+IN1, R10.2
- removed net N$18: IC2.OUT2, R13.1, R15.2, R16.1
- removed net N$19: C10.1, IC2.+IN2, R14.2
- new net N$16: IC1.-RG, IC2C.+IN, R7.2
- new net N$17: D2.AC, IC2C.-IN, IC2C.OUT, R3.2, R8.1
- new net N$23: IC2A.-IN, R11.1, R12.2
- net +5V: now also IC2P.V+; no longer IC2.+VS
- net -5V: now also IC2P.V-; no longer IC2.-VS
- net N$10: now also IC2B.-IN, R16.1, R17.2; no longer D4.AC, IC2.-IN4, IC2.OUT4, R4.2, R9.1
- net N$14: now also C8.1, IC2A.+IN, R10.2; no longer IC2.-IN1, R11.2, R12.2
- net N$22: now also C10.1, IC2B.+IN, R14.2; no longer IC2.-IN2, R16.2, R17.2
- net N$7: now also D4.AC, IC2D.-IN, IC2D.OUT, R4.2, R9.1; no longer IC1.-RG, IC2.+IN3, R7.2
- net N$8: now also IC2D.+IN; no longer IC2.+IN4
- net N$9: now also IC2B.OUT, R13.1, R15.2, R16.2; no longer D2.AC, IC2.-IN3, IC2.OUT3, R3.2, R8.1
- net OUT: now also IC2A.OUT, R11.2; no longer IC2.OUT1, R11.1
Other:
- moved on the sheet: C10, C11, C5, C6, C7, C8, C9, IC1, JP1, R10, R11, R12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

Commit message: Better comps
Parts:
- removed IN+, IN-: 1503_09, con-lumberg:1503_09
- added +IN, -IN: (no value), SparkFun-Connectors:AUDIO-JACKSMD
- C1, C10, C11, C2, C3, C8, C9: device rcl:C-EUC0805 -> SparkFun-Passives:CAP0805
- C4, C5, C6, C7: value 0.1uF -> 100nF; device rcl:C-EUC0805 -> SparkFun-Passives:CAP0805
- R1, R10, R11, R12, R13, R14, R15, R16, R17, R2, R3, R4, R5, R6, R7, R8, R9: device rcl:R-EU_R0805 -> SparkFun-Passives:RESISTOR0805-RES
Connections:
- net GND: now also +IN.SLEEVE, -IN.SLEEVE; no longer IN+.1, IN-.1
- net N$1: now also -IN.LEFT; no longer IN-.2
- net N$11: now also C10.1; no longer C11.2
- net N$2: now also -IN.RIGHT; no longer IN-.3
- net N$22: now also C11.2; no longer C10.1
- net N$3: now also +IN.LEFT, R1.1; no longer IN+.3, R3.1
- net N$4: now also +IN.RIGHT, R3.1; no longer IN+.2, R1.1
Other:
- moved on the sheet: C10, C11

Commit message: .
Parts:
- removed D3, D4: BAV199, diode:BAV199
- +IN, -IN: value (none) -> AUDIOJACK2.5-SMD; device SparkFun-Connectors:AUDIO-JACKSMD -> femtoexg:AUDIOJACK2.5-SMD
- D1: device diode:BAV199 -> SparkFun-DiscreteSemi:BAV99; PROD_ID (none) -> DIO-10647
- D2: device diode:BAV199 -> SparkFun-DiscreteSemi:BAV99
Connections:
- net +5V: now also D1.C2, D2.C2; no longer D1.C, D2.C, D3.C, D4.C
- net -5V: now also D1.A1, D2.A1; no longer D1.A, D2.A, D3.A, D4.A
- net GND: now also +IN.GND1, +IN.GND2, +IN.SW, -IN.GND1, -IN.GND2, -IN.SW; no longer +IN.SLEEVE, -IN.SLEEVE
- net N$17: no longer D2.AC
- net N$5: now also D2.COM; no longer D3.AC
- net N$6: now also D1.COM; no longer D1.AC
- net N$7: no longer D4.AC
Other:
- moved on the sheet: C1, C3, IC2D, R2, R4, R6, R9

Commit message: Amp routing
Connections:
- net N$10: now also IC2A.-IN; no longer IC2B.-IN
- net N$14: now also IC2B.+IN; no longer IC2A.+IN
- net N$16: now also IC2D.+IN; no longer IC2C.+IN
- net N$17: now also IC2D.-IN, IC2D.OUT; no longer IC2C.-IN, IC2C.OUT
- net N$22: now also IC2A.+IN; no longer IC2B.+IN
- net N$23: now also IC2B.-IN; no longer IC2A.-IN
- net N$7: now also IC2C.-IN, IC2C.OUT; no longer IC2D.-IN, IC2D.OUT
- net N$8: now also IC2C.+IN; no longer IC2D.+IN
- net N$9: now also IC2A.OUT; no longer IC2B.OUT
- net OUT: now also IC2B.OUT; no longer IC2A.OUT
Other:
- moved on the sheet: IC2A, IC2B, IC2C, IC2D
Changed lines of the file:
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@@
 <instance part="JP1" gate="A" x="431.8" y="-10.16"/>
 <instance part="GND15" gate="1" x="408.94" y="-5.08" rot="R270"/>
-<instance part="IC2" gate="A" x="309.88" y="-5.08"/>
-<instance part="IC2" gate="B" x="241.3" y="-5.08"/>
-<instance part="IC2" gate="C" x="111.76" y="10.16" rot="R180"/>
-<instance part="IC2" gate="D" x="111.76" y="-50.8" rot="R180"/>
+<instance part="IC2" gate="A" x="241.3" y="-5.08"/>
+<instance part="IC2" gate="B" x="309.88" y="-5.08"/>
+<instance part="IC2" gate="C" x="111.76" y="-50.8" rot="R180"/>
+<instance part="IC2" gate="D" x="111.76" y="10.16" rot="R180"/>
 <instance part="IC2" gate="P" x="360.68" y="-5.08"/>
 <instance part="R1" gate="G$1" x="20.32" y="27.94"/>
@@
 <wire x1="127" y1="-53.34" x2="127" y2="-12.7" width="0.1524" layer="91"/>
 <junction x="127" y="-12.7"/>
-<pinref part="IC2" gate="D" pin="+IN"/>
+<pinref part="R7" gate="G$1" pin="1"/>
+<pinref part="IC2" gate="C" pin="+IN"/>
 <wire x1="119.38" y1="-53.34" x2="127" y2="-53.34" width="0.1524" layer="91"/>
-<pinref part="R7" gate="G$1" pin="1"/>
 </segment>
 </net>
@@
 <wire x1="314.96" y1="-15.24" x2="320.04" y2="-15.24" width="0.1524" layer="91"/>
 <wire x1="320.04" y1="-15.24" x2="320.04" y2="-5.08" width="0.1524" layer="91"/>
-<pinref part="IC2" gate="A" pin="OUT"/>
-<wire x1="320.04" y1="-5.08" x2="317.5" y2="-5.08" width="0.1524" layer="91"/>
 <wire x1="320.04" y1="5.08" x2="320.04" y2="-5.08" width="0.1524" layer="91"/>
 <junction x="320.04" y="-5.08"/>
@@
 <pinref part="R11" gate="G$1" pin="2"/>
 <pinref part="C9" gate="G$1" pin="2"/>
+<pinref part="IC2" gate="B" pin="OUT"/>
+<wire x1="317.5" y1="-5.08" x2="320.04" y2="-5.08" width="0.1524" layer="91"/>
 </segment>
 </net>
@@
 <wire x1="127" y1="2.54" x2="127" y2="7.62" width="0.1524" layer="91"/>
 <wire x1="127" y1="7.62" x2="134.62" y2="7.62" width="0.1524" layer="91"/>
+<pinref part="R7" gate="G$1" pin="2"/>
+<pinref part="IC2" gate="D" pin="+IN"/>
+<wire x1="119.38" y1="7.62" x2="127" y2="7.62" width="0.1524" layer="91"/>
 <junction x="127" y="7.62"/>
-<wire x1="119.38" y1="7.62" x2="127" y2="7.62" width="0.1524" layer="91"/>
-<pinref part="IC2" gate="C" pin="+IN"/>
-<pinref part="R7" gate="G$1" pin="2"/>
 </segment>
 </net>
@@
 <wire x1="25.4" y1="20.32" x2="91.44" y2="20.32" width="0.1524" layer="91"/>
 <wire x1="121.92" y1="20.32" x2="121.92" y2="12.7" width="0.1524" layer="91"/>
-<pinref part="IC2" gate="C" pin="-IN"/>
-<wire x1="121.92" y1="12.7" x2="119.38" y2="12.7" width="0.1524" layer="91"/>
-<pinref part="IC2" gate="C" pin="OUT"/>
-<wire x1="104.14" y1="10.16" x2="101.6" y2="10.16" width="0.1524" layer="91"/>
 <wire x1="101.6" y1="10.16" x2="101.6" y2="20.32" width="0.1524" layer="91"/>
 <junction x="101.6" y="20.32"/>
@@
 <pinref part="R3" gate="G$1" pin="2"/>
 <pinref part="R8" gate="G$1" pin="1"/>
+<pinref part="IC2" gate="D" pin="-IN"/>
+<wire x1="119.38" y1="12.7" x2="121.92" y2="12.7" width="0.1524" layer="91"/>
+<pinref part="IC2" gate="D" pin="OUT"/>
+<wire x1="104.14" y1="10.16" x2="101.6" y2="10.16" width="0.1524" layer="91"/>
 </segment>
 </net>
@@
 <wire x1="101.6" y1="-40.64" x2="121.92" y2="-40.64" width="0.1524" layer="91"/>
 <wire x1="121.92" y1="-40.64" x2="121.92" y2="-48.26" width="0.1524" layer="91"/>
-<pinref part="IC2" gate="D" pin="-IN"/>
-<wire x1="121.92" y1="-48.26" x2="119.38" y2="-48.26" width="0.1524" layer="91"/>
-<pinref part="IC2" gate="D" pin="OUT"/>
-<wire x1="104.14" y1="-50.8" x2="101.6" y2="-50.8" width="0.1524" layer="91"/>
 <wire x1="101.6" y1="-50.8" x2="101.6" y2="-40.64" width="0.1524" layer="91"/>
 <junction x="101.6" y="-40.64"/>
@@
 <pinref part="R4" gate="G$1" pin="2"/>
 <pinref part="R9" gate="G$1" pin="1"/>
+<pinref part="IC2" gate="C" pin="OUT"/>
+<wire x1="104.14" y1="-50.8" x2="101.6" y2="-50.8" width="0.1524" layer="91"/>
+<pinref part="IC2" gate="C" pin="-IN"/>
+<wire x1="119.38" y1="-48.26" x2="121.92" y2="-48.26" width="0.1524" layer="91"/>
 </segment>
 </net>
@@
 <wire x1="246.38" y1="-15.24" x2="251.46" y2="-15.24" width="0.1524" layer="91"/>
 <wire x1="251.46" y1="-15.24" x2="251.46" y2="-5.08" width="0.1524" layer="91"/>
-<pinref part="IC2" gate="B" pin="OUT"/>
-<wire x1="251.46" y1="-5.08" x2="248.92" y2="-5.08" width="0.1524" layer="91"/>
+<wire x1="251.46" y1="-5.08" x2="251.46" y2="-2.54" width="0.1524" layer="91"/>
 <wire x1="246.38" y1="5.08" x2="251.46" y2="5.08" width="0.1524" layer="91"/>
 <wire x1="251.46" y1="5.08" x2="251.46" y2="-2.54" width="0.1524" layer="91"/>
-<junction x="251.46" y="-5.08"/>
-<wire x1="251.46" y1="-2.54" x2="251.46" y2="-5.08" width="0.1524" layer="91"/>
 <wire x1="264.16" y1="-2.54" x2="251.46" y2="-2.54" width="0.1524" layer="91"/>
 <junction x="251.46" y="-2.54"/>
@@
 <pinref part="R15" gate="G$1" pin="2"/>
 <pinref part="R16" gate="G$1" pin="2"/>
+<pinref part="IC2" gate="A" pin="OUT"/>
+<wire x1="248.92" y1="-5.08" x2="251.46" y2="-5.08" width="0.1524" layer="91"/>
+<junction x="251.46" y="-5.08"/>
 </segment>
 </net>
@@
 <wire x1="236.22" y1="-15.24" x2="231.14" y2="-15.24" width="0.1524" layer="91"/>
 <wire x1="231.14" y1="-15.24" x2="231.14" y2="-7.62" width="0.1524" layer="91"/>
-<pinref part="IC2" gate="B" pin="-IN"/>
-<wire x1="231.14" y1="-7.62" x2="233.68" y2="-7.62" width="0.1524" layer="91"/>
 <wire x1="231.14" y1="-17.78" x2="231.14" y2="-15.24" width="0.1524" layer="91"/>
 <junction x="231.14" y="-15.24"/>
 <pinref part="R17" gate="G$1" pin="2"/>
 <pinref part="R16" gate="G$1" pin="1"/>
+<pinref part="IC2" gate="A" pin="-IN"/>
+<wire x1="233.68" y1="-7.62" x2="231.14" y2="-7.62" width="0.1524" layer="91"/>
 </segment>
 </net>
@@
 <segment>
 <wire x1="223.52" y1="-17.78" x2="223.52" y2="-2.54" width="0.1524" layer="91"/>
-<pinref part="IC2" gate="B" pin="+IN"/>
-<wire x1="223.52" y1="-2.54" x2="233.68" y2="-2.54" width="0.1524" layer="91"/>
 <wire x1="220.98" y1="-2.54" x2="223.52" y2="-2.54" width="0.1524" layer="91"/>
-<junction x="223.52" y="-2.54"/>
 <pinref part="R14" gate="G$1" pin="2"/>
 <pinref part="C11" gate="G$1" pin="2"/>
+<pinref part="IC2" gate="A" pin="+IN"/>
+<wire x1="233.68" y1="-2.54" x2="223.52" y2="-2.54" width="0.1524" layer="91"/>
+<junction x="223.52" y="-2.54"/>
 </segment>
 </net>
@@
 <segment>
 <wire x1="299.72" y1="-17.78" x2="299.72" y2="-15.24" width="0.1524" layer="91"/>
-<pinref part="IC2" gate="A" pin="-IN"/>
 <wire x1="299.72" y1="-15.24" x2="299.72" y2="-7.62" width="0.1524" layer="91"/>
-<wire x1="299.72" y1="-7.62" x2="302.26" y2="-7.62" width="0.1524" layer="91"/>
 <wire x1="304.8" y1="-15.24" x2="299.72" y2="-15.24" width="0.1524" layer="91"/>
 <junction x="299.72" y="-15.24"/>
 <pinref part="R11" gate="G$1" pin="1"/>
 <pinref part="R12" gate="G$1" pin="2"/>
+<pinref part="IC2" gate="B" pin="-IN"/>
+<wire x1="302.26" y1="-7.62" x2="299.72" y2="-7.62" width="0.1524" layer="91"/>
 </segment>
 </net>
@@
 <segment>
 <wire x1="292.1" y1="-19.05" x2="292.1" y2="-2.54" width="0.1524" layer="91"/>
-<pinref part="IC2" gate="A" pin="+IN"/>
-<wire x1="292.1" y1="-2.54" x2="302.26" y2="-2.54" width="0.1524" layer="91"/>
 <wire x1="289.56" y1="-2.54" x2="292.1" y2="-2.54" width="0.1524" layer="91"/>
-<junction x="292.1" y="-2.54"/>
 <pinref part="R10" gate="G$1" pin="2"/>
 <pinref part="C8" gate="G$1" pin="1"/>
+<pinref part="IC2" gate="B" pin="+IN"/>
+<wire x1="302.26" y1="-2.54" x2="292.1" y2="-2.54" width="0.1524" layer="91"/>
+<junction x="292.1" y="-2.54"/>
 </segment>
 </net>
@@
 </sheet>
 </sheets>
-<errors>
-</errors>
 </schematic>
 </drawing>
